File: Kicad Files/EEG kicad/EEG2.kicad_sch (KiCad schematic)
At the start: 503 parts, among them J2 GPIO_CONNECTOR, U1 INA823, U10 LF357, U100 LF357, U101 MCP4161, U102 LF357, U103 LF357, U104 LF357, U105 LF357, U106 LF357, U107 LF357, U108 MCP4161, U109 LF357, U11 LF357, U110 INA823, U111 INA823, U112 LF357, U113 MCP4161, U114 LF357, U115 LF357, U116 LF357, U117 LF357, U118 LF357, U119 LF357, U12 LF357, U120 MCP4161, U121 LF357, U122 INA823, U13 MCP4161, U14 LF357, U15 INA823, U16 LF357, U17 LF357, U18 LF357, U19 MCP4161, U2 LF357, U20 LF357, U21 INA823, U22 LF357, U23 LF357, U24 LF357, U25 MCP4161, U26 LF357, U27 INA823, U28 LF357, U29 LF357, U3 LF357, U30 LF357, U31 MCP4161, U32 LF357, U33 LF357, U34 MCP4161, U35 LF357, U36 LF357, U37 LF357, U38 LF357, U39 LF357, U4 LF357, U40 LF357, U41 MCP4161, U42 LF357, U43 INA823, U44 INA823, U45 LF357, U46 MCP4161, U47 LF357, U48 LF357, U49 LF357, U5 MCP4161, U50 LF357, U51 LF357, U52 LF357, U53 MCP4161, U54 LF357, U55 INA823, U56 INA823, U57 LF357, U58 MCP4161, U59 LF357, U6 LF357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

Commit message: Schematic Errors Fixed, some footprints done
Parts:
- removed C1, C103, C105, C106, C110, C112, C12, C14, C15, C19, C21, C22, C26, C28, C29, C33, C35, C5, C7, C78, C8, C82, C84, C85, C89, C91, C92, C96, C98, C99: 0.22uF, symbol Device:C
- removed C10, C100, C101, C102, C107, C108, C109, C11, C16, C17, C18, C2, C23, C24, C25, C3, C30, C31, C32, C4, C79, C80, C81, C86, C87, C88, C9, C93, C94, C95: 1uF, symbol Device:C
- removed C104, C111, C13, C20, C27, C34, C6, C83, C90, C97: 2uF, symbol Device:C
- removed J2: GPIO_CONNECTOR, lib:PinSocket_2x20_P2.54mm_Vertical_Centered_Anchor, symbol Connector_Generic:Conn_02x20_Odd_Even
- removed R1, R13, R133, R145, R157, R169, R181, R25, R37, R49: 1000, symbol Device:R
- removed R10, R142, R154, R166, R178, R190, R22, R34, R46, R58: 1.5k, symbol Device:R
- removed R11, R139, R143, R151, R155, R163, R167, R175, R179, R187, R19, R191, R23, R31, R35, R43, R47, R55, R59, R7: 1k, symbol Device:R
- removed R12, R144, R156, R168, R180, R192, R24, R36, R48, R60: 100, symbol Device:R
- removed R134, R135, R14, R146, R147, R15, R158, R159, R170, R171, R182, R183, R2, R26, R27, R3, R38, R39, R50, R51: 3k, symbol Device:R
- removed R136, R137, R138, R148, R149, R150, R16, R160, R161, R162, R17, R172, R173, R174, R18, R184, R185, R186, R28, R29, R30, R4, R40, R41, R42, R5, R52, R53, R54, R6: 10k, symbol Device:R
- removed R140, R152, R164, R176, R188, R20, R32, R44, R56, R8: 1K, symbol Device:R
- removed R141, R153, R165, R177, R189, R21, R33, R45, R57, R9: 150k, symbol Device:R
- removed U1, U15, U21, U27, U69, U75, U81, U87, U9, U93: INA823, Package_SO:VSSOP-8_3x3mm_P0.65mm, symbol Amplifier_Instrumentation:INA333xxDGK
- removed U10, U11, U12, U14, U16, U17, U18, U2, U20, U22, U23, U24, U26, U28, U29, U3, U30, U32, U4, U6, U70, U71, U73, U74, U76, U77, U79, U80, U82, U83, U85, U86, U88, U89, U91, U92, U94, U95, U97, U98: LF357, symbol Amplifier_Operational:LF357
- removed U13, U19, U25, U31, U5, U72, U78, U84, U90, U96: MCP4161, Package_DIP:DIP-8_W7.62mm_Socket, symbol Potentiometer_Digital:MCP4161-xxxx-P
- removed U7: Teensy4.1, symbol teensy:Teensy4.1
- added J1: Conn_01x05_Pin, Connector_PinHeader_1.27mm:PinHeader_1x05_P1.27mm_Vertical, symbol Connector:Conn_01x05_Pin
- added J2: Conn_01x11_Pin, Connector_PinHeader_1.27mm:PinHeader_1x11_P1.27mm_Vertical, symbol Connector:Conn_01x11_Pin
- C113, C117, C118, C121, C122, C126, C127, C131, C132, C135, C136, C140, C36, C40, C41, C44, C45, C49, C50, C54, C55, C58, C59, C63, C64, C68, C69, C72, C73, C77: footprint (none) -> Capacitor_SMD:C_0603_1608Metric
- C114, C115, C116, C123, C124, C125, C128, C129, C130, C137, C138, C139, C37, C38, C39, C46, C47, C48, C51, C52, C53, C60, C61, C62, C65, C66, C67, C74, C75, C76: footprint (none) -> Capacitor_SMD:C_0805_2012Metric
- U100, U102, U103, U104, U105, U106, U107, U109, U112, U114, U115, U116, U117, U118, U119, U121, U33, U35, U36, U37, U38, U39, U40, U42, U45, U47, U48, U49, U50, U51, U52, U54, U57, U59, U60, U61, U62, U63, U64, U66: value LF357 -> LF356N
Connections:
- net GND: now also C117.2, C118.2, C121.2, C122.2, C131.2, C132.2, C135.2, C136.2, C40.2, C41.2, C44.2, C45.2, C54.2, C58.2, C68.2, C69.2, C72.2, C73.2, R101.2, R105.2, R112.2, R116.2, R118.2, R123.2, R125.2, R129.2, R196.2, R200.2, R202.2, R207.2, R209.2, R213.2, R220.2, R224.2, R226.2, R231.2, R233.2, R237.2, R64.2, R68.2, R70.2, R75.2, R77.2, R81.2, R99.2, U101.4 (V_{SS}), U101.5 (P0A), U108.4 (V_{SS}), U108.5 (P0A), U110.5 (Ref), U111.5 (Ref), U113.4 (V_{SS}), U113.5 (P0A), U120.4 (V_{SS}), U120.5 (P0A), U122.5 (Ref), U34.4 (V_{SS}), U34.5 (P0A), U41.4 (V_{SS}), U41.5 (P0A), U43.5 (Ref), U44.5 (Ref), U53.4 (V_{SS}), U53.5 (P0A), U55.5 (Ref), U56.5 (Ref), U58.4 (V_{SS}), U58.5 (P0A), U65.4 (V_{SS}), U65.5 (P0A), U67.5 (Ref), U68.1 (GND), U8.5 (Ref), U99.5 (Ref), J1.5 (Pin_5)
- net GPIO14_TXD0: now also J1.2 (Pin_2)
- net GPIO15_RXD0: now also J1.1 (Pin_1)
- net Vss: now reaches U100.4 (V-), U102.4 (V-), U103.4 (V-), U104.4 (V-), U105.4 (V-), U106.4 (V-), U107.4 (V-), U109.4 (V-), U110.4 (V-), U115.4 (V-), U117.4 (V-), U119.4 (V-), U121.4 (V-), U122.4 (V-), U33.4 (V-), U35.4 (V-), U36.4 (V-), U37.4 (V-), U38.4 (V-), U39.4 (V-), U40.4 (V-), U42.4 (V-), U43.4 (V-), U44.4 (V-), U45.4 (V-), U47.4 (V-), U48.4 (V-), U49.4 (V-), U50.4 (V-), U51.4 (V-), U52.4 (V-), U54.4 (V-), U55.4 (V-), U56.4 (V-), U57.4 (V-), U59.4 (V-), U61.4 (V-), U63.4 (V-), U8.4 (V-), U99.4 (V-)
- net Vss: now also J1.4 (Pin_4)
- net Vdd: now reaches U100.7 (V+), U101.8 (V_{DD}), U102.7 (V+), U103.7 (V+), U104.7 (V+), U105.7 (V+), U106.7 (V+), U107.7 (V+), U108.8 (V_{DD}), U109.7 (V+), U110.7 (V+), U111.7 (V+), U112.7 (V+), U113.8 (V_{DD}), U114.7 (V+), U115.7 (V+), U116.7 (V+), U117.7 (V+), U118.7 (V+), U119.7 (V+), U120.8 (V_{DD}), U121.7 (V+), U122.7 (V+), U33.7 (V+), U34.8 (V_{DD}), U35.7 (V+), U36.7 (V+), U37.7 (V+), U38.7 (V+), U39.7 (V+), U40.7 (V+), U41.8 (V_{DD}), U42.7 (V+), U43.7 (V+), U44.7 (V+), U45.7 (V+), U46.8 (V_{DD}), U47.7 (V+), U48.7 (V+), U49.7 (V+), U50.7 (V+), U51.7 (V+), U52.7 (V+), U53.8 (V_{DD}), U54.7 (V+), U55.7 (V+), U56.7 (V+), U57.7 (V+), U58.8 (V_{DD}), U59.7 (V+), U60.7 (V+), U61.7 (V+), U62.7 (V+), U63.7 (V+), U64.7 (V+), U65.8 (V_{DD}), U66.7 (V+), U67.7 (V+), U8.7 (V+), U99.7 (V+)
- net Vdd: now also C60.1, U46.6 (P0W), U50.6, J1.3 (Pin_3); no longer C39.1, U37.6, U41.6 (P0W)
- net Ref_Electrode: now reaches U111.2 (-)
- net Ref_Electrode: now also U110.2 (-), U122.2 (-), U43.2 (-), U44.2 (-), U55.2 (-), U56.2 (-), U67.2 (-), U8.2 (-), U99.2 (-), J2.11 (Pin_11)
- net Electrode5: now reaches U111.3 (+)
- net Electrode5: now also J2.5 (Pin_5)
- net Electrode1: now reaches U8.3 (+)
- net Electrode1: now also J2.1 (Pin_1)
- net Electrode8: now reaches U67.3 (+)
- net Electrode8: now also J2.8 (Pin_8)
- net Electrode3: now reaches U56.3 (+)
- net Electrode3: now also J2.3 (Pin_3)
- net Electrode10: now reaches U122.3 (+)
- net Electrode10: now also J2.10 (Pin_10)
- net Electrode4: now reaches U99.3 (+)
- net Electrode4: now also J2.4 (Pin_4)
- net Electrode9: now reaches U110.3 (+)
- net Electrode9: now also J2.9 (Pin_9)
- net Electrode7: now reaches U55.3 (+)
- net Electrode7: now also J2.7 (Pin_7)
- net Electrode6: now reaches U43.3 (+)
- net Electrode6: now also J2.6 (Pin_6)
- net Electrode2: now reaches U44.3 (+)
- net Electrode2: now also J2.2 (Pin_2)
- new net: C39.1, U37.6, U41.6 (P0W)
- no-connect marks 293 -> 103
Other:
- note removed: "August Nguyen"
- note removed: "Teensy TX2 (Pin 30) → RX of USB-to-Serial adapter Teensy RX2 (Pin 31) → TX of USB-to-Serial adapter"
- moved on the sheet: C113, C114, C115, C116, C117, C118, C119, C120, C121, C122, C123, C124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

Commit message: EEG
Connections:
- net at U101.2 (SCK), U108.2 (SCK), U113.2 (SCK)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: now also U58.1 (~{CS}), U68.11 (9_OUT1C)
Changed lines of the file:
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@@
 	)
 	(junction
+		(at 266.7 246.38)
+		(diameter 0)
+		(color 0 0 0 0)
+	)
+	(junction
 		(at 377.19 279.4)
 		(diameter 0)
@@
 	)
 	(junction
+		(at 271.78 246.38)
+		(diameter 0)
+		(color 0 0 0 0)
+	)
+	(junction
 		(at 332.74 279.4)
 		(diameter 0)
@@
 	(wire
 		(pts
-			(xy 279.4 246.38) (xy 266.7 246.38)
+			(xy 279.4 246.38) (xy 271.78 246.38)
 		)
 		(stroke
@@
 	(wire
 		(pts
+			(xy 271.78 246.38) (xy 271.78 245.11)
+		)
+		(stroke
+			(width 0)
+			(type default)
+		)
+	)
+	(wire
+		(pts
 			(xy 278.13 340.36) (xy 271.78 340.36)
 		)
@@
 	(wire
 		(pts
-			(xy 276.86 358.14) (xy 276.86 353.06)
+			(xy 271.78 246.38) (xy 271.78 293.37)
 		)
 		(stroke
@@
 	(wire
 		(pts
-			(xy 234.95 245.11) (xy 234.95 246.38)
+			(xy 276.86 358.14) (xy 276.86 353.06)
 		)
 		(stroke
@@
 	(wire
 		(pts
+			(xy 271.78 246.38) (xy 266.7 246.38)
+		)
+		(stroke
+			(width 0)
+			(type default)
+		)
+	)
+	(wire
+		(pts
 			(xy 35.56 340.36) (xy 35.56 339.09)
 		)
@@
 	(wire
 		(pts
-			(xy 234.95 245.11) (xy 271.78 245.11)
+			(xy 234.95 246.38) (xy 266.7 246.38)
 		)
 		(stroke
@@
 		)
 		(stroke
-			(width 0)
-			(type default)
-		)
-	)
-	(wire
-		(pts
-			(xy 271.78 245.11) (xy 271.78 293.37)
-		)
-		(stroke

Commit message: Add files via upload
Parts:
- removed C113, C117, C118, C121, C122, C126, C127, C131, C132, C135, C136, C140, C54, C55, C58, C59, C63, C64, C68, C69, C72, C73, C77: 0.22uF, Capacitor_SMD:C_0603_1608Metric, symbol Device:C
- removed C114, C115, C116, C123, C124, C125, C128, C129, C130, C137, C138, C139, C51, C52, C53, C60, C61, C62, C65, C66, C67, C74, C75, C76: 1uF, Capacitor_SMD:C_0805_2012Metric, symbol Device:C
- removed C119, C120, C133, C134, C56, C57, C70, C71: 2uF, symbol Device:C
- removed R100, R117, R124, R201, R208, R225, R232, R69, R76, R93: 1.5k, symbol Device:R
- removed R101, R116, R119, R122, R125, R200, R203, R206, R209, R224, R227, R230, R233, R68, R71, R74, R77, R92, R95, R98: 1k, symbol Device:R
- removed R102, R103, R104, R113, R114, R115, R126, R127, R128, R197, R198, R199, R210, R211, R212, R221, R222, R223, R234, R235, R236, R65, R66, R67, R78, R79, R80, R89, R90, R91: 10k, symbol Device:R
- removed R105, R112, R129, R196, R213, R220, R237, R64, R81, R88: 100, symbol Device:R
- removed R106, R107, R110, R111, R130, R131, R194, R195, R214, R215, R218, R219, R238, R239, R62, R63, R82, R83, R86, R87: 3k, symbol Device:R
- removed R108, R109, R132, R193, R216, R217, R240, R61, R84, R85: 1000, symbol Device:R
- removed R118, R123, R202, R207, R226, R231, R70, R75, R94, R99: 150k, symbol Device:R
- removed R120, R121, R204, R205, R228, R229, R72, R73, R96, R97: 1K, symbol Device:R
- removed U100, U102, U103, U104, U105, U106, U107, U109, U112, U114, U115, U116, U117, U118, U119, U121, U33, U35, U36, U37, U38, U39, U40, U42, U45, U47, U48, U49, U50, U51, U52, U54, U57, U59, U60, U61, U62, U63, U64, U66: LF356N, symbol Amplifier_Operational:LF357
- removed U101, U108, U113, U120, U34, U41, U46, U53, U58, U65: MCP4161, Package_DIP:DIP-8_W7.62mm_Socket, symbol Potentiometer_Digital:MCP4161-xxxx-P
- removed U110, U111, U122, U43, U44, U55, U56, U67, U8, U99: INA823, Package_SO:VSSOP-8_3x3mm_P0.65mm, symbol Amplifier_Instrumentation:INA333xxDGK
- removed U68: Teensy4.1, symbol teensy:Teensy4.1
- added C1, C10, C14, C143, C144, C145, C146, C147, C15, C16, C17, C18, C19, C2, C20, C27, C28, C29, C3, C30, C31, C35, C7, C8, C85, C86, C87, C88, C89, C9, C94, C96, C97, C98, C99: 1uF, Capacitor_SMD:C_0805_2012Metric, symbol Device:C
- added C100, C101, C102, C103, C104, C105, C106, C107, C108, C109, C11, C110, C111, C112, C12, C13, C141, C142, C21, C22, C23, C24, C25, C26, C32, C33, C34, C4, C5, C6: 0.22uF, Capacitor_SMD:C_0603_1608Metric, symbol Device:C
- added R1, R10, R13, R145, R146, R147, R148, R149, R166, R168, R170, R173, R176, R18, R185, R186, R187, R188, R189, R190, R191, R192, R21, R22, R242, R243, R25, R26, R34, R36, R41, R42, R43, R44, R49, R54, R57, R58, R6, R9: 1k, symbol Device:R
- added R11, R171, R174, R177, R178, R179, R180, R181, R182, R183, R184, R19, R20, R23, R241, R244, R245, R246, R247, R37, R38, R39, R40, R45, R46, R55, R56, R59, R7, R8: 10k, symbol Device:R
- added R12, R24, R248, R249, R250, R251, R252, R47, R48, R60: 150k, symbol Device:R
- added R14, R150, R151, R152, R154, R156, R16, R160, R161, R162, R163, R164, R2, R27, R28, R31, R32, R4, R50, R52: 2652, symbol Device:R
- added R15, R153, R155, R157, R158, R159, R29, R3, R30, R51: 1326, symbol Device:R
- added R165, R167, R169, R17, R172, R175, R33, R35, R5, R53: 100, symbol Device:R
- added U1, U124, U125, U126, U127, U128, U14, U25, U26, U32: AD5293, Package_SO:TSSOP-14_4.4x5mm_P0.65mm, symbol Potentiometer_Digital:AD5293
- added U10, U11, U12, U123, U13, U17, U18, U19, U20, U21, U22, U23, U24, U28, U29, U3, U30, U31, U4, U5, U6, U80, U81, U82, U83, U84, U85, U86, U87, U88, U89, U90, U91, U92, U93, U94, U95, U96, U97, U98: LF356N, symbol Amplifier_Operational:LF357
- added U15, U16, U2, U27, U75, U76, U77, U78, U79, U9: INA823, Package_SO:VSSOP-8_3x3mm_P0.65mm, symbol Amplifier_Instrumentation:INA333xxDGK
- added U7: Teensy4.1, EEG Project:Teensy41, symbol teensy:Teensy4.1
- C36, C40, C41, C44, C45, C49, C50: value 0.22uF -> 1uF; footprint Capacitor_SMD:C_0603_1608Metric -> Capacitor_SMD:C_0805_2012Metric
- C42, C43: value 2uF -> 1uF; footprint (none) -> Capacitor_SMD:C_0805_2012Metric
Connections:
- net Electrode1: now also U2.3 (+)
- net Electrode10: now also U75.3 (+)
- net Electrode2: now also U9.3 (+)
- net Electrode3: now also U15.3 (+)
- net Electrode4: now also U16.3 (+)
- net Electrode5: now also U27.3 (+)
- net Electrode6: now also U79.3 (+)
- net Electrode7: now also U78.3 (+)
- net Electrode8: now also U77.3 (+)
- net Electrode9: now also U76.3 (+)
- net GND: now also C100.2, C101.2, C103.2, C105.2, C107.2, C11.2, C110.2, C111.2, C112.2, C13.2, C141.2, C142.2, C21.2, C22.2, C25.2, C26.2, C32.2, C34.2, C4.2, C6.2, R10.2, R12.2, R166.2, R168.2, R170.2, R173.2, R176.2, R18.2, R186.2, R188.2, R190.2, R192.2, R22.2, R24.2, R243.2, R248.2, R249.2, R250.2, R251.2, R252.2, R34.2, R36.2, R42.2, R44.2, R47.2, R48.2, R54.2, R58.2, R6.2, R60.2, U1.2 (Vss-), U1.5 (RL), U1.9 (GND), U10.4 (V-), U11.4 (V-), U12.4 (V-), U123.4 (V-), U124.2 (Vss-), U124.5 (RL), U124.9 (GND), U125.2 (Vss-), U125.5 (RL), U125.9 (GND), U126.2 (Vss-), U126.5 (RL), U126.9 (GND), U127.2 (Vss-), U127.5 (RL), U127.9 (GND), U128.2 (Vss-), U128.5 (RL), U128.9 (GND), U13.4 (V-), U14.2 (Vss-), U14.5 (RL), U14.9 (GND), U15.4 (V-), U15.5 (Ref), U16.4 (V-), U16.5 (Ref), U17.4 (V-), U18.4 (V-), U19.4 (V-), U2.4 (V-), U2.5 (Ref), U20.4 (V-), U21.4 (V-), U22.4 (V-), U23.4 (V-), U24.4 (V-), U25.2 (Vss-), U25.5 (RL), U25.9 (GND), U26.2 (Vss-), U26.5 (RL), U26.9 (GND), U27.4 (V-), U27.5 (Ref), U28.4 (V-), U29.4 (V-), U3.4 (V-), U30.4 (V-), U31.4 (V-), U32.2 (Vss-), U32.5 (RL), U32.9 (GND), U4.4 (V-), U5.4 (V-), U6.4 (V-), U75.4 (V-), U75.5 (Ref), U76.4 (V-), U76.5 (Ref), U77.4 (V-), U77.5 (Ref), U78.4 (V-), U78.5 (Ref), U79.4 (V-), U79.5 (Ref), U80.4 (V-), U81.4 (V-), U82.4 (V-), U83.4 (V-), U84.4 (V-), U85.4 (V-), U86.4 (V-), U87.4 (V-), U88.4 (V-), U89.4 (V-), U9.4 (V-), U9.5 (Ref), U90.4 (V-), U91.4 (V-), U92.4 (V-), U93.4 (V-), U94.4 (V-), U95.4 (V-), U96.4 (V-), U97.4 (V-), U98.4 (V-); no longer C40.2, C41.2, C44.2, C45.2
- net GPIO14_TXD0: now also U7.26 (34_RX8)
- net GPIO15_RXD0: now also U7.27 (35_TX8)
- net Ref_Electrode: now also U15.2 (-), U16.2 (-), U2.2 (-), U27.2 (-), U75.2 (-), U76.2 (-), U77.2 (-), U78.2 (-), U79.2 (-), U9.2 (-)
- net Vss: now also U1.6 (Vdd+), U1.8 (Vlog), U10.7 (V+), U11.7 (V+), U12.7 (V+), U123.7 (V+), U124.6 (Vdd+), U124.8 (Vlog), U125.6 (Vdd+), U125.8 (Vlog), U126.6 (Vdd+), U126.8 (Vlog), U127.6 (Vdd+), U127.8 (Vlog), U128.6 (Vdd+), U128.8 (Vlog), U13.7 (V+), U14.6 (Vdd+), U14.8 (Vlog), U15.7 (V+), U16.7 (V+), U17.7 (V+), U18.7 (V+), U19.7 (V+), U2.7 (V+), U20.7 (V+), U21.7 (V+), U22.7 (V+), U23.7 (V+), U24.7 (V+), U25.6 (Vdd+), U25.8 (Vlog), U26.6 (Vdd+), U26.8 (Vlog), U27.7 (V+), U28.7 (V+), U29.7 (V+), U3.7 (V+), U30.7 (V+), U31.7 (V+), U32.6 (Vdd+), U32.8 (Vlog), U4.7 (V+), U5.7 (V+), U6.7 (V+), U75.7 (V+), U76.7 (V+), U77.7 (V+), U78.7 (V+), U79.7 (V+), U80.7 (V+), U81.7 (V+), U82.7 (V+), U83.7 (V+), U84.7 (V+), U85.7 (V+), U86.7 (V+), U87.7 (V+), U88.7 (V+), U89.7 (V+), U9.7 (V+), U90.7 (V+), U91.7 (V+), U92.7 (V+), U93.7 (V+), U94.7 (V+), U95.7 (V+), U96.7 (V+), U97.7 (V+), U98.7 (V+)
- net at C49.1: now also C50.1, R150.1, R160.2
- net at C49.2: now also C50.2, R153.2, U80.2 (-), U80.6
- net at C39.1: now also C18.1, R30.2, U19.2 (-), U19.6
- net at C37.1: now also C9.1, R15.2, U10.2 (-), U10.6
- net at C38.1: now also C17.1, R29.2, U17.2 (-), U17.6; no longer C37.2
- net at C41.1: now also C42.1, R156.1, R164.2
- net at C46.1: now also C45.1, R152.1, R162.2
- net at C48.1: now also C47.1, R151.1, R161.2
- net at C48.2: now also C47.2, R155.2, U82.2 (-), U82.6; no longer C47.1
- net at C38.2: now also C17.2, R27.1, R31.2
- net at C40.1: now also C30.1, R51.2, U28.2 (-), U28.6
- net at C36.1: now also C2.1, R3.2, U3.2 (-), U3.6
- net at C43.2: now also C44.2, R158.2, U86.2 (-), U86.6
- net at C46.2: now also C45.2, R157.2, U84.2 (-), U84.6
- net at C36.2: now also C2.2, R2.1, R4.2
- net at C39.2: now also C18.2, R28.1, R32.2
- net at C43.1: now also C44.1, R154.1, R163.2
- net at C42.2: now also C41.2, R159.2, U88.2 (-), U88.6
- new net: C106.1, R189.1, R245.1, U92.6
- new net: C106.2, R177.2, R182.1
- new net: C89.1, R156.2, U79.6
- new net: C31.2, R52.1, U29.3 (+)
- new net: C30.2, C40.2, R50.1, R52.2
- new net: R17.1, R19.1, U11.2 (-), U11.6
- new net: R17.2, R18.1, U10.3 (+)
- new net: C99.2, R164.1, U89.3 (+)
- new net: C141.1, R246.2, U98.3 (+)
- new net: C1.1, R2.2, U2.6
- new net: C104.1, R187.1, R244.1, U91.6
- new net: R187.2, R188.1, U91.2 (-)
- new net: C147.1, U123.6, U128.4 (RW)
- new net: C147.2, R252.1, U7.40 (18_A4_SDA)
- new net: C88.2, C98.1, R158.1
- new net: C98.2, R163.1, U87.3 (+)
- new net: C10.1, C8.2, R15.1
- new net: U1.10 (SDI), U124.10 (SDI), U125.10 (SDI), U126.10 (SDI), U127.10 (SDI), U128.10 (SDI), U14.10 (SDI), U25.10 (SDI), U26.10 (SDI), U32.10 (SDI), U7.13 (11_MOSI_CTX1)
- new net: U1.11 (CLK), U124.11 (CLK), U125.11 (CLK), U126.11 (CLK), U127.11 (CLK), U128.11 (CLK), U14.11 (CLK), U25.11 (CLK), U26.11 (CLK), U32.11 (CLK), U7.35 (13_SCK_LED)
- new net: U26.12 (~{CS}), U7.7 (5_IN2)
- new net: U24.2 (-), U26.3 (RH)
- new net: C28.1, U24.6, U26.4 (RW)
- new net: C15.2, C19.1, R29.1
- new net: C5.1, R11.1, R9.1, U5.6
- new net: C5.2, R7.2, R8.1
- new net: R185.2, R186.1, U90.2 (-)
- new net: C100.1, R180.2, U90.3 (+)
- new net: C102.1, R185.1, R241.1, U90.6
- new net: R13.1, U9.1 (Rg)
- new net: C8.1, R14.2, U9.6
- new net: R13.2, U9.8 (Rg)
- new net: C109.1, R242.1, R247.1, U94.6
- new net: C109.2, R179.2, R184.1
- new net: R167.2, R168.1, U82.3 (+)
- new net: R147.1, U77.1 (Rg)
- new net: C87.1, R152.2, U77.6
- new net: R147.2, U77.8 (Rg)
- new net: C16.2, C20.1, R30.1
- new net: R25.1, U15.1 (Rg)
- new net: C15.1, R27.2, U15.6
- new net: R25.2, U15.8 (Rg)
- new net: R167.1, R174.1, U83.2 (-), U83.6
- new net: C96.2, R161.1, U83.3 (+)
- new net: U126.3 (RH), U97.2 (-)
- new net: C112.1, R245.2, U97.3 (+)
- new net: C145.1, U126.4 (RW), U97.6
- new net: C14.2, R24.1, U7.42 (20_A6_TX5_LRCLK1)
- new net: R53.1, R55.1, U29.2 (-), U29.6
- new net: C86.1, R151.2, U76.6
- new net: C86.2, C96.1, R155.1
- new net: R57.2, R58.1, U30.2 (-)
- new net: C33.1, R57.1, R59.1, U30.6
- new net: C34.1, R59.2, U31.3 (+)
- new net: R5.1, R7.1, U4.2 (-), U4.6
- new net: C3.2, R4.1, U4.3 (+)
- new net: R148.1, U78.1 (Rg)
- new net: C88.1, R154.2, U78.6
- new net: R148.2, U78.8 (Rg)
- new net: R21.2, R22.1, U12.2 (-)
- new net: C11.1, R20.2, U12.3 (+)
- new net: C12.1, R21.1, R23.1, U12.6
- new net: C19.2, R31.1, U18.3 (+)
- new net: U124.3 (RH), U95.2 (-)
- new net: C110.1, R241.2, U95.3 (+)
- new net: C143.1, U124.4 (RW), U95.6
- new net: R5.2, R6.1, U3.3 (+)
- new net: C10.2, R16.1, U11.3 (+)
- new net: C37.2, C9.2, R14.1, R16.2
- new net: U23.2 (-), U25.3 (RH)
- new net: C25.1, R45.2, U23.3 (+)
- new net: C27.1, U23.6, U25.4 (RW)
- new net: C23.1, R41.1, R45.1, U21.6
- new net: C23.2, R37.2, R39.1
- new net: C108.1, R191.1, R246.1, U93.6
- new net: C108.2, R178.2, R183.1
- new net: R165.1, R171.1, U81.2 (-), U81.6
- new net: C102.2, R171.2, R180.1
- new net: C35.1, U31.6, U32.4 (RW)
- new net: C35.2, R60.1, U7.45 (23_A9_CRX1_MCLK1)
- new net: R149.1, U79.1 (Rg)
- new net: R149.2, U79.8 (Rg)
- new net: R175.2, R176.1, U88.3 (+)
- new net: C85.2, C94.1, R153.1
- new net: C94.2, R160.1, U81.3 (+)
- new net: U127.3 (RH), U98.2 (-)
- new net: C146.1, U127.4 (RW), U98.6
- new net: U128.12 (~{CS}), U7.14 (12_MISO_MQSL)
- new net: U123.2 (-), U128.3 (RH)
- new net: U124.12 (~{CS}), U7.9 (7_RX2_OUT1A)
- new net: R175.1, R179.1, U89.2 (-), U89.6
- new net: R41.2, R42.1, U21.2 (-)
- new net: C21.1, R39.2, U21.3 (+)
- new net: C1.2, C3.1, R3.1
- new net: C29.1, R50.2, U27.6
- new net: C29.2, C31.1, R51.1
- new net: U14.12 (~{CS}), U7.5 (3_LRCLK2)
- new net: U13.2 (-), U14.3 (RH)
- new net: C14.1, U13.6, U14.4 (RW)
- new net: C12.2, R19.2, R20.1
- new net: R169.1, R177.1, U85.2 (-), U85.6
- new net: C97.2, R162.1, U85.3 (+)
- new net: R242.2, R243.1, U94.2 (-)
- new net: R10.1, R9.2, U5.2 (-)
- new net: C4.1, R8.2, U5.3 (+)
- new net: C20.2, R32.1, U20.3 (+)
- new net: C24.1, R43.1, R46.1, U22.6
- new net: C24.2, R38.2, R40.1
- new net: C28.2, R48.1, U7.44 (22_A8_CTX1)
- new net: C27.2, R47.1, U7.43 (21_A7_RX5_BCLK1)
- new net: U127.12 (~{CS}), U7.12 (10_CS_MQSR)
- new net: C33.2, R55.2, R56.1
- new net: C7.2, R12.1, U7.41 (19_A5_SCL)
- new net: C145.2, R250.1, U7.38 (16_A2_RX4_SCL1)
- new net: U32.12 (~{CS}), U7.8 (6_OUT1D)
- new net: U31.2 (-), U32.3 (RH)
- new net: R35.1, R38.1, U20.2 (-), U20.6
- new net: C146.2, R251.1, U7.39 (17_A3_TX4_SDA1)
- new net: R145.1, U75.1 (Rg)
- new net: C85.1, R150.2, U75.6
- new net: R145.2, U75.8 (Rg)
- new net: R169.2, R170.1, U84.3 (+)
- new net: R191.2, R192.1, U93.2 (-)
- new net: C104.2, R174.2, R181.1
- new net: R33.2, R34.1, U17.3 (+)
- new net: C26.1, R46.2, U24.3 (+)
- new net: R33.1, R37.1, U18.2 (-), U18.6
- new net: C101.1, R181.2, U91.3 (+)
- new net: C107.1, R184.2, U94.3 (+)
- new net: C89.2, C99.1, R159.1
- new net: C87.2, C97.1, R157.1
- new net: R43.2, R44.1, U22.2 (-)
- new net: C22.1, R40.2, U22.3 (+)
- new net: C142.1, R247.2, U123.3 (+)
- new net: R165.2, R166.1, U80.3 (+)
- new net: C144.1, U125.4 (RW), U96.6
- new net: C144.2, R249.1, U7.37 (15_A1_RX3_SPDIF_IN)
- new net: C143.2, R248.1, U7.36 (14_A0_TX3_SPDIF_OUT)
- new net: R26.1, U16.1 (Rg)
- new net: R26.2, U16.8 (Rg)
- new net: C105.1, R183.2, U93.3 (+)
- new net: C6.1, R11.2, U6.3 (+)
- new net: R189.2, R190.1, U92.2 (-)
- new net: C111.1, R244.2, U96.3 (+)
- new net: C32.1, R56.2, U30.3 (+)
- new net: R53.2, R54.1, U28.3 (+)
- new net: R1.1, U2.1 (Rg)
- new net: R1.2, U2.8 (Rg)
- new net: C103.1, R182.2, U92.3 (+)
- new net: R172.1, R178.1, U87.2 (-), U87.6
- new net: U25.12 (~{CS}), U7.6 (4_BCLK2)
- new net: R35.2, R36.1, U19.3 (+)
- new net: R172.2, R173.1, U86.3 (+)
- new net: C7.1, U1.4 (RW), U6.6
- new net: R49.1, U27.1 (Rg)
- new net: R49.2, U27.8 (Rg)
- new net: C16.1, R28.2, U16.6
- new net: R146.1, U76.1 (Rg)
- new net: R146.2, U76.8 (Rg)
- new net: C13.1, R23.2, U13.3 (+)
- new net: U125.12 (~{CS}), U7.10 (8_TX2_IN1)
- new net: U125.3 (RH), U96.2 (-)
- new net: U1.12 (~{CS}), U7.4 (2_OUT2)
- new net: U1.3 (RH), U6.2 (-)
- new net: U126.12 (~{CS}), U7.11 (9_OUT1C)
- no-connect marks 103 -> 144
Other:
- moved on the sheet: J1, J2
