File: Kicad Files/EEG kicad/EEG2.kicad_pcb (KiCad board)
At the start: 2 copper layers, 108 x 130.8 mm, 273 parts, among them J1 Conn_02x20_Top_Bottom, J2 Conn_01x05_Pin, U1 INA823, U10 LF356M, U11 LF356M, U12 LF356M, U13 LF356M, U14 LF356M, U15 LF356M, U16 LF356M, U17 LF356M, U18 LF356M, U19 LF356M, U2 INA823, U20 LF356M, U21 LF356M, U22 LF356M, U23 LF356M, U24 LF356M, U25 LF356M, U26 AD5293, U27 AD5293, U28 AD5293, U29 AD5293, U3 INA823, U30 AD5293, U31 Teensy4.1, U32 AD5293, U33 AD5293, U34 AD5293, U35 AD5293, U36 AD5293, U37 LF356M, U38 LF356M, U39 LF356M, U4 INA823, U40 LF356M, U41 LF356M, U42 LF356M, U43 LF356M, U44 LF356M, U45 LF356M, U46 LF356M, U47 LF356M, U48 LF356M, U49 LF356M, U5 INA823, U50 LF356M, U51 LF356M, U52 LF356M, U53 LF356M, U54 LF356M, U55 LF356M, U56 LF356M, U57 INA823, U58 INA823, U59 INA823, U6 LF356M, U60 INA823, U61 INA823, U7 LF356M, U8 LF356M, U9 LF356M

Commit message: EEG Done and some rearrangements
Parts:
- added G***: LOGO, logo:logo_HorizontalText, B.Cu at (154.9, 115.6)

Commit message: AR & EEG corrected
Parts:
- J2: value Conn_01x05_Pin -> Conn_01x04_Pin; footprint Connector_PinHeader_1.27mm:PinHeader_1x05_P1.27mm_Vertical -> Connector_PinHeader_1.27mm:PinHeader_1x04_P1.27mm_Vertical
- moved C58 117.4 mm to (172.2, 25.6)
- moved C60 117.4 mm to (176.1, 25.6)
- moved C71 117.4 mm to (152.0, 32.8)
- moved C75 117.4 mm to (156.1, 32.8)
- moved R109 117.4 mm to (168.8, 31.9)
- moved R115 117.4 mm to (156.1, 29.4)
- moved R125 117.4 mm to (152.0, 29.4)
- moved R70 117.4 mm to (203.2, 25.6)
- moved R90 117.4 mm to (179.6, 25.6)
- moved U36 117.4 mm to (203.1, 29.4)
- moved U41 117.4 mm to (190.4, 29.4)
- moved U46 117.4 mm to (175.2, 29.4)
- moved U55 117.4 mm to (163.8, 33.3)
- moved C45 117.4 mm to (196.8, 28.1)
- moved C50 117.4 mm to (183.6, 30.7)
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Connections:
- J2 pad 3: Vdd -> Vss
- J2 pad 4: Vss -> GND
- U31 pad 10: unconnected-(U31-8_TX2_IN1-Pad10) -> CS 4
- U31 pad 11: unconnected-(U31-9_OUT1C-Pad11) -> CS 3
- U31 pad 12: unconnected-(U31-10_CS_MQSR-Pad12) -> CS 2
- U31 pad 4: unconnected-(U31-2_OUT2-Pad4) -> CS 10
- U31 pad 5: unconnected-(U31-3_LRCLK2-Pad5) -> CS 9
- U31 pad 6: unconnected-(U31-4_BCLK2-Pad6) -> CS 8
- U31 pad 7: unconnected-(U31-5_IN2-Pad7) -> CS 7
- U31 pad 8: unconnected-(U31-6_OUT1D-Pad8) -> CS 6
- U31 pad 9: unconnected-(U31-7_RX2_OUT1A-Pad9) -> CS 5
Routing:
- net CLK: track 0.00 -> 180.3 mm, vias 0 -> 10
- net SDI: track 0.00 -> 151.5 mm, vias 0 -> 10
- net Electrode Output 1: track 6.03 -> 110.0 mm
- net CS 1: track 0.00 -> 92.2 mm, vias 0 -> 2
- net Electrode Output 2: track 6.03 -> 95.6 mm
- net CS 2: track 0.00 -> 83.4 mm, vias 0 -> 2
- net Electrode Output 3: track 6.03 -> 84.9 mm
- net CS 3: track 0.00 -> 73.4 mm, vias 0 -> 2
- net Electrode Output 4: track 6.03 -> 74.5 mm
- net CS 4: track 0.00 -> 64.9 mm, vias 0 -> 2
- net Electrode Output 5: track 6.03 -> 62.7 mm
- net CS 5: track 0.00 -> 54.3 mm, vias 0 -> 2
- net Electrode Output 6: track 6.03 -> 56.7 mm
- net CS 6: track 0.00 -> 42.5 mm, vias 0 -> 2
- net Electrode Output 7: track 6.03 -> 47.0 mm
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Other:
- outline, holes or cut-outs redrawn

Commit message: work
Parts:
- moved G*** 53.3 mm to (156.2, 113.0)
- moved R109 5.28 mm to (168.9, 26.7), turned to 0 degrees
- moved R106 5.20 mm to (169.4, 58.0), turned to 90 degrees
- moved R108 5.10 mm to (168.9, 45.0), turned to 90 degrees
- moved R105 5.08 mm to (168.9, 52.8), turned to 0 degrees
- moved R107 5.08 mm to (168.9, 39.9), turned to 0 degrees
- moved R110 4.89 mm to (168.9, 31.8), turned to 90 degrees
- turned C63 to 0 degrees
- turned C65 to 0 degrees
- turned C69 to 0 degrees
- turned C70 to 0 degrees
- turned C72 to 0 degrees
- turned C74 to 0 degrees
Routing:
- net Ref_Electrode: track 0.00 -> 152.7 mm, vias 0 -> 1
- net Net-(U6--): track 124.1 -> 20.7 mm, vias 12 -> 2
- net Net-(C10-Pad2): track 60.5 -> 10.1 mm
- net Electrode10: track 0.00 -> 42.6 mm
- net Electrode1: track 0.00 -> 42.3 mm
- net Net-(U6-+): track 49.6 -> 12.4 mm
- net Electrode9: track 0.00 -> 35.4 mm
- net Electrode2: track 0.00 -> 34.5 mm
- net Electrode8: track 0.00 -> 27.4 mm
- net Net-(U52--): track 0.00 -> 27.2 mm, vias 0 -> 2
- net Electrode3: track 0.00 -> 26.4 mm
- net Net-(U56--): track 0.00 -> 24.8 mm, vias 0 -> 2
- net Net-(U48--): track 0.00 -> 20.7 mm, vias 0 -> 2
- net Net-(U54--): track 0.00 -> 20.7 mm, vias 0 -> 2
- net Net-(U50--): track 0.00 -> 20.7 mm, vias 0 -> 2
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Other:
- outline, holes or cut-outs redrawn

Commit message: work..
Parts:
- moved R65 0.77 mm to (202.7, 91.4)
Routing:
- net Vss: track 0.00 -> 255.7 mm
- net Net-(U56--): track 24.8 -> 20.6 mm
- net Net-(C71-Pad1): track 11.1 -> 13.1 mm, vias 0 -> 2
- net Electrode Output 5: track 62.7 -> 64.4 mm, vias 0 -> 2
- net CLK: track 180.3 -> 178.6 mm
- net Electrode Output 1: track 110.0 -> 111.4 mm, vias 0 -> 1
- net CS 8: track 24.3 -> 23.2 mm
- net Electrode Output 2: track 95.6 -> 96.6 mm, vias 0 -> 2
- net Electrode Output 8: track 39.4 -> 40.4 mm, vias 0 -> 2
- net Net-(U36-RH): track 15.8 -> 14.9 mm
- net Net-(U55-+): track 9.98 -> 10.7 mm, vias 0 -> 2
- net Net-(C80-Pad1): track 7.26 -> 7.86 mm, vias 0 -> 2
- net Electrode Output 7: track 47.0 -> 47.4 mm, vias 0 -> 2
- net Electrode Output 9: track 34.9 -> 35.0 mm, vias 0 -> 2
- net Electrode Output 6: vias 0 -> 2
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
Commit message: EEG done
Routing:
- net Vss: track 255.7 -> 980.6 mm
- net GND: track 0.00 -> 319.3 mm, vias 0 -> 132
- net Net-(U42-+): track 5.20 -> 14.0 mm, vias 0 -> 2
- net Net-(U43-+): track 5.20 -> 14.0 mm, vias 0 -> 2
- net Net-(U46-+): track 5.20 -> 13.8 mm, vias 0 -> 2
- net Net-(U44-+): track 5.20 -> 13.4 mm, vias 0 -> 2
- net Net-(U45-+): track 5.20 -> 13.4 mm, vias 0 -> 2
- net Net-(C27-Pad2): track 9.55 -> 11.9 mm, vias 0 -> 2
- net Net-(U18--): track 10.6 -> 12.3 mm, vias 0 -> 2
- net Net-(U22--): track 15.8 -> 14.6 mm
- net Net-(U23--): track 15.8 -> 14.7 mm
- net Net-(U32-RH): track 15.8 -> 14.7 mm
- net Net-(U35-RH): track 15.8 -> 14.7 mm
- net Net-(U34-RH): track 15.8 -> 14.7 mm
- net Net-(U33-RH): track 15.8 -> 14.7 mm
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- added copper zone on B.Cu, net GND
- added copper zone on F.Cu, net GND
