File: Kicad Files/Old/EEG kicad — no golden fingers/EEG2.kicad_sch (KiCad schematic)
At the start: 263 parts, among them J1 Conn_01x05_Pin, J2 Conn_01x11_Pin, U1 AD5293, U10 LF356N, U11 LF356N, U12 LF356N, U123 LF356N, U124 AD5293, U125 AD5293, U126 AD5293, U127 AD5293, U128 AD5293, U13 LF356N, U14 AD5293, U15 INA823, U16 INA823, U17 LF356N, U18 LF356N, U19 LF356N, U2 INA823, U20 LF356N, U21 LF356N, U22 LF356N, U23 LF356N, U24 LF356N, U25 AD5293, U26 AD5293, U27 INA823, U28 LF356N, U29 LF356N, U3 LF356N, U30 LF356N, U31 LF356N, U32 AD5293, U4 LF356N, U5 LF356N, U6 LF356N, U7 Teensy4.1, U75 INA823, U76 INA823, U77 INA823, U78 INA823, U79 INA823, U80 LF356N, U81 LF356N, U82 LF356N, U83 LF356N, U84 LF356N, U85 LF356N, U86 LF356N, U87 LF356N, U88 LF356N, U89 LF356N, U9 INA823, U90 LF356N, U91 LF356N, U92 LF356N, U93 LF356N, U94 LF356N, U95 LF356N, U96 LF356N, U97 LF356N, U98 LF356N

Commit message: EEG new PCB done
Parts:
- U7: footprint EEG Project:Teensy41 -> Teensy 4.1:Teensy41
Changed lines of the file:
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@@
 			)
 		)
-		(property "Footprint" "EEG Project:Teensy41"
+		(property "Footprint" "Teensy 4.1:Teensy41"
 			(at 170.18 279.4 0)
 			(effects
