File: Kicad Files/EEG/Mother/Mother.kicad_pcb (KiCad board)
At the start: 2 copper layers, 66 x 116.8 mm, 13 parts, among them J1 Conn_01x05_Pin, U1 Teensy4.1

Commit message: Gerber generated
Parts:
- removed the G*** at (124.5, 110.5)
- added G***: LOGO, logo:logo_HorizontalText, B.Cu at (104.1, 129.5)
