File: Kicad Files/AR Glass/Glass.kicad_sch (KiCad schematic)
At the start: 6 parts, among them U1 Pico, U2 OLED Driver, U3 OLED Driver 2, U4 Camera

Commit message: AR revised
Parts:
- removed U2: OLED Driver, Connector_PinHeader_2.54mm:PinHeader_1x07_P2.54mm_Vertical, symbol AR_Library:OLD Driver
- removed U3: OLED Driver 2, Connector_PinHeader_2.54mm:PinHeader_1x07_P2.54mm_Vertical, symbol AR_Library:OLD Driver
- added J1, J2: Conn_01x07_Pin, Connector_PinHeader_2.54mm:PinHeader_1x07_P2.54mm_Vertical, symbol Connector:Conn_01x07_Pin
- added TP4, TP5, TP6, TP7: TestPoint, Connector_PinHeader_2.54mm:PinHeader_1x01_P2.54mm_Vertical, symbol Connector:TestPoint
- added U2, U3: OLED Driver, Connector_PinHeader_2.54mm:PinHeader_1x07_P2.54mm_Vertical, symbol AR_Library:OLED Driver
Connections:
- net +3.3V: now also J1.1 (Pin_1), J2.1 (Pin_1), TP5.1, TP7.1, U2.1 (VCC), U3.1 (VCC)
- net GND: now also J1.2 (Pin_2), J2.2 (Pin_2), TP4.1, TP6.1, U2.2 (GND), U3.2 (GND)
- net GP13: now also J1.5 (Pin_5), U2.5 (CS)
- net GP14: now also J1.7 (Pin_7), U2.7 (RST)
- net GP15: now also J1.6 (Pin_6), U2.6 (DC)
- net GP2: now also J1.4 (Pin_4), J2.4 (Pin_4), U2.4 (CLK), U3.4 (CLK)
- net GP3: now also J1.3 (Pin_3), J2.3 (Pin_3), U2.3 (DIN), U3.3 (DIN)
- net GP5: now also J2.5 (Pin_5), U3.5 (CS)
- net GP6: now also J2.7 (Pin_7), U3.7 (RST)
- net GP7: now also J2.6 (Pin_6), U3.6 (DC)
- no-connect marks 0 -> 19
