File: Kicad Files/AR Glass/Glass.kicad_sch (KiCad schematic)
At the start: 12 parts, among them J1 OLED1, J2 OLED2, J3 Camera1, J4 OLED1, J5 OLED2, U1 Pico

Commit message: some changes
Parts:
- added J6: Camera2, Connector_FFC-FPC:Molex_54548-1071_1x10-1MP_P0.5mm_Horizontal, symbol Connector:Conn_01x08_Pin
Connections:
- net 3.3V is gone; now on net +3.3V: J1.1 (Pin_1), J2.1 (Pin_1), J4.1 (Pin_1), J5.1 (Pin_1)
- net CLK_Cam is gone; now on net CLK_LED: U1.4 (GPIO2)
- net CS_Cam1 is gone; now on net CS_LED1: U1.17 (GPIO13)
- net CS_Cam2 is gone; now on net CS_LED2: U1.7 (GPIO5)
- net DC_Cam1 is gone; now on net DC_LED1: U1.20 (GPIO15)
- net DC_Cam2 is gone; now on net DC_LED2: U1.10 (GPIO7)
- net DIN_Cam is gone; now on net DIN_LED: U1.5 (GPIO3)
- net GP10 is gone; now on net DO_Cam1: U1.14 (GPIO10)
- net GP16 is gone; now on net VSYNC_Cam1: U1.21 (GPIO16)
- net GP18 is gone; now on net PCLK_Cam1: U1.24 (GPIO18)
- net GP19 is gone; now on net HREF_Cam1: U1.25 (GPIO19)
- net GP20 is gone; now on net SDA_Cam1: U1.26 (GPIO20)
- net RST_Cam1 is gone; now on net RST_LED1: U1.19 (GPIO14)
- net RST_Cam2 is gone; now on net RST_LED2: U1.9 (GPIO6)
- net SCL_Cam1 is gone; now on net SCL_Cam: J3.2 (Pin_2)
- net +3.3V: now also J6.1 (Pin_1)
- net GND: now also J6.8 (Pin_8)
- net VSYNC_Cam2: now reaches U1.11 (GPIO8)
- net VSYNC_Cam2: now also J6.4 (Pin_4)
- net HREF_Cam2: now reaches U1.12 (GPIO9)
- net HREF_Cam2: now also J6.5 (Pin_5)
- net PCLK_Cam2: now reaches U1.15 (GPIO11)
- net PCLK_Cam2: now also J6.6 (Pin_6)
- net DO_Cam2: now reaches U1.16 (GPIO12)
- net DO_Cam2: now also J6.7 (Pin_7)
- net SDA_Cam2: now reaches U1.6 (GPIO4)
- net SDA_Cam2: now also J6.3 (Pin_3)
- net GP21 renamed SCL_Cam
- net SCL_Cam: now also J6.2 (Pin_2)
- no-connect marks 19 -> 14
