File: Kicad Files/AR Glass/Glass.kicad_pcb (KiCad board)
At the start: 2 copper layers, 74.3 x 89.3 mm, 23 parts, among them J1 Conn_01x07_Pin, J2 Conn_01x07_Pin, U1 Pico, U2 OLED Driver, U3 OLED Driver, U4 Camera

Commit message: EEG Done and some rearrangements
Routing:
- removed copper zone on B.Cu, net GND
- removed copper zone on F.Cu, net GND
Changed lines of the file:
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@@
 		(net 50)
 	)
-	(zone
-		(net 3)
-		(net_name "GND")
-		(layers "F&B.Cu")
-		(hatch edge 0.5)
-		(connect_pads
-			(clearance 0.5)
-		)
-		(min_thickness 0.25)
-		(filled_areas_thickness no)
-		(fill yes
-			(thermal_gap 0.5)
-			(thermal_bridge_width 0.5)
-		)
-		(polygon
-			(pts
-				(xy 102.87 27.94) (xy 102.87 124.46) (xy 187.96 124.46) (xy 186.69 26.67)
-			)
-		)
-	)
 )

Commit message: AR modified
Parts:
- removed the REF** at (177.2, 99.9)
- removed the REF** at (177.2, 75.8)
- removed the REF** at (177.2, 113.9)
- removed the REF** at (177.2, 89.8)
- added REF**: MountingHole_2.2mm_M2, MountingHole:MountingHole_2.2mm_M2, F.Cu at (156.3, 69.2)
- added REF**: MountingHole_2.2mm_M2, MountingHole:MountingHole_2.2mm_M2, F.Cu at (214.0, 69.2)
- added REF**: MountingHole_2.2mm_M2, MountingHole:MountingHole_2.2mm_M2, F.Cu at (156.3, 94.5)
- added REF**: MountingHole_2.2mm_M2, MountingHole:MountingHole_2.2mm_M2, F.Cu at (214.0, 94.5)
- moved G*** 45.1 mm to (186.7, 80.7)
- moved REF** 45.1 mm to (195.6, 83.2)
- moved TP7 45.1 mm to (213.4, 78.8)
- moved J1 45.1 mm to (208.9, 73.9)
- moved TP6 45.1 mm to (213.4, 83.5)
- moved G*** 20.9 mm to (129.0, 81.9)
- moved J2 20.9 mm to (151.2, 74.3)
- moved REF** 20.9 mm to (137.9, 83.8)
- moved TP4 20.9 mm to (155.6, 84.8)
- moved TP5 20.9 mm to (155.6, 79.9)
- moved REF** 1.20 mm to (174.0, 57.8)
- moved U2 0.89 mm to (175.9, 38.1)
- moved TP2 0.86 mm to (114.9, 58.4)
- moved REF** 0.58 mm to (174.0, 33.5)
Routing:
- net GND: track 63.1 -> 70.9 mm, vias 10 -> 14
- net GP14: track 9.42 -> 16.7 mm
- net GP15: track 11.8 -> 8.28 mm
- net GP13: track 16.6 -> 17.6 mm
- net GP3: track 72.9 -> 73.8 mm
- net GP2: track 75.5 -> 76.4 mm
- net 3.3V: track 93.7 -> 93.2 mm
- added copper zone on B.Cu, net GND
- added copper zone on F.Cu, net GND
Other:
- board size 74.3 x 89.3 mm -> 111.2 x 67.3 mm

Commit message: AR & EEG corrected
Parts:
- removed the REF** at (156.3, 69.2)
- removed the REF** at (214.0, 69.2)
- removed the REF** at (174.0, 33.5)
- removed the REF** at (156.3, 94.5)
- removed the REF** at (214.0, 94.5)
- removed the REF** at (174.0, 57.8)
- added REF**: MountingHole_2mm, MountingHole:MountingHole_2mm, F.Cu at (109.2, 97.7)
- added REF**: MountingHole_2mm, MountingHole:MountingHole_2mm, F.Cu at (174.0, 65.4)
- added REF**: MountingHole_2mm, MountingHole:MountingHole_2mm, F.Cu at (109.2, 59.7)
- added REF**: MountingHole_2mm, MountingHole:MountingHole_2mm, F.Cu at (174.0, 59.7)
- added REF**: MountingHole_2mm, MountingHole:MountingHole_2mm, F.Cu at (174.0, 92.0)
- added REF**: MountingHole_2mm, MountingHole:MountingHole_2mm, F.Cu at (174.0, 97.7)
- added REF**: MountingHole_2mm, MountingHole:MountingHole_2mm, F.Cu at (109.2, 92.0)
- added REF**: MountingHole_2mm, MountingHole:MountingHole_2mm, F.Cu at (174.0, 124.4)
- added REF**: MountingHole_2mm, MountingHole:MountingHole_2mm, F.Cu at (109.2, 124.4)
- added REF**: MountingHole_2mm, MountingHole:MountingHole_2mm, F.Cu at (174.0, 33.0)
- added REF**: MountingHole_2mm, MountingHole:MountingHole_2mm, F.Cu at (109.2, 33.0)
- added REF**: MountingHole_2mm, MountingHole:MountingHole_2mm, F.Cu at (109.2, 65.4)
- 3.3 V: renamed from TP5
- 3.3 V: renamed from TP3
- 3.3 V: renamed from TP7
- moved 3.3 V 49.5 mm to (173.4, 107.9)
- moved REF** 49.5 mm to (155.6, 112.4)
- moved G*** 49.5 mm to (146.8, 109.8)
- moved GND 49.5 mm to (173.4, 112.6)
- moved J1 49.5 mm to (169.0, 103.1)
- moved G*** 18.1 mm to (146.8, 78.7)
- moved J2 18.1 mm to (169.0, 71.1)
- moved 3.3 V 18.1 mm to (173.4, 76.7)
- moved GND 18.1 mm to (173.4, 81.5)
- moved REF** 18.1 mm to (155.6, 80.6)
- renumbered TP6 to GND, TP2 to GND, TP4 to GND
Routing:
- net GP13: track 17.6 -> 20.6 mm
Other:
- board size 111.2 x 67.3 mm -> 72.4 x 96.5 mm
- board text added: "3.3V"
- board text added: "GND"
- board text added: "GP10"
- board text added: "GP16"
- board text added: "GP18"
- board text added: "GP19"
- board text added: "GP20"
- board text added: "GP21"

Commit message: work
Parts:
- removed 3.3 V: TestPoint, Connector_PinHeader_2.54mm:PinHeader_1x01_P2.54mm_Vertical (x3)
- removed the G*** at (146.8, 109.8)
- removed the G*** at (146.8, 78.7)
- removed GND (x3): TestPoint, Connector_PinHeader_2.54mm:PinHeader_1x01_P2.54mm_Vertical
- removed REF** (x12): MountingHole_2mm, MountingHole:MountingHole_2mm
- removed REF** (x2): OLED Driver, MCU_RaspberryPi_and_Boards:OLED Driver
- removed U2, U3: OLED Driver, Connector_PinHeader_2.54mm:PinHeader_1x07_P2.54mm_Vertical
- removed U4: Camera, Connector_PinHeader_2.54mm:PinHeader_1x08_P2.54mm_Vertical
- added J3: Camera1, Connector_FFC-FPC:Molex_54548-1071_1x10-1MP_P0.5mm_Horizontal, F.Cu at (108.0, 54.1)
- added J4: OLED1, Connector_FFC-FPC:Molex_54548-1071_1x10-1MP_P0.5mm_Horizontal, F.Cu at (70.8, 39.1)
- added J5: OLED2, Connector_FFC-FPC:Molex_54548-1071_1x10-1MP_P0.5mm_Horizontal, F.Cu at (74.1, 56.1)
- added TP1: TestPoint, Connector_PinHeader_2.54mm:PinHeader_1x01_P2.54mm_Vertical, F.Cu at (88.5, 48.7)
- added TP2: TestPoint, Connector_PinHeader_2.54mm:PinHeader_1x01_P2.54mm_Vertical, F.Cu at (88.5, 53.3)
- added TP3: TestPoint, Connector_PinHeader_2.54mm:PinHeader_1x01_P2.54mm_Vertical, F.Cu at (93.1, 48.7)
- added TP4: TestPoint, Connector_PinHeader_2.54mm:PinHeader_1x01_P2.54mm_Vertical, F.Cu at (93.1, 53.3)
- added TP5: TestPoint, Connector_PinHeader_2.54mm:PinHeader_1x01_P2.54mm_Vertical, F.Cu at (97.8, 48.7)
- added TP6: TestPoint, Connector_PinHeader_2.54mm:PinHeader_1x01_P2.54mm_Vertical, F.Cu at (97.8, 53.3)
- J1: value Conn_01x07_Pin -> OLED1; footprint Connector_PinHeader_2.54mm:PinHeader_1x07_P2.54mm_Vertical -> Connector_FFC-FPC:Molex_54548-1071_1x10-1MP_P0.5mm_Horizontal
- J2: value Conn_01x07_Pin -> OLED2; footprint Connector_PinHeader_2.54mm:PinHeader_1x07_P2.54mm_Vertical -> Connector_FFC-FPC:Molex_54548-1071_1x10-1MP_P0.5mm_Horizontal
- moved J1 88.4 mm to (107.7, 39.4), turned to 90 degrees
- moved J2 83.4 mm to (94.5, 33.4)
Connections:
- J1 pad 3: GP3 -> DIN_LED
- J1 pad 4: GP2 -> CLK_LED
- J1 pad 5: GP13 -> CS_LED1
- J1 pad 6: GP15 -> DC_LED1
- J1 pad 7: GP14 -> RST_LED1
- J2 pad 3: GP3 -> DIN_LED
- J2 pad 4: GP2 -> CLK_LED
- J2 pad 5: GP5 -> CS_LED2
- J2 pad 6: GP7 -> DC_LED2
- J2 pad 7: GP6 -> RST_LED2
- U1 pad 10: GP7 -> DC_Cam2
- U1 pad 17: GP13 -> CS_Cam1
- U1 pad 19: GP14 -> RST_Cam1
- U1 pad 20: GP15 -> DC_Cam1
- U1 pad 36: 3.3V -> +3.3V
- U1 pad 4: GP2 -> CLK_Cam
- U1 pad 5: GP3 -> DIN_Cam
- U1 pad 7: GP5 -> CS_Cam2
- U1 pad 9: GP6 -> RST_Cam2
Routing:
- net 3.3V: track 93.2 -> 0.00 mm
- net GP2: track 76.4 -> 0.00 mm
- net GP3: track 73.8 -> 0.00 mm
- net CLK_Cam: track 0.00 -> 64.4 mm
- net DIN_Cam: track 0.00 -> 56.8 mm
- net /GP21: track 46.8 -> 3.59 mm
- net +3.3V: track 0.00 -> 42.6 mm
- net GP7: track 38.7 -> 0.00 mm
- net GP6: track 31.0 -> 0.00 mm
- net DC_Cam2: track 0.00 -> 28.1 mm
- net GP5: track 27.7 -> 0.00 mm, vias 1 -> 0
- net GND: track 70.9 -> 43.6 mm, vias 14 -> 8
- net RST_Cam2: track 0.00 -> 24.3 mm
- net CS_Cam2: track 0.00 -> 23.2 mm, vias 0 -> 1
- net GP13: track 20.6 -> 0.00 mm
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- removed copper zone on B.Cu, net GND
- removed copper zone on F.Cu, net GND
Other:
- board size 72.4 x 96.5 mm -> 72.4 x 31.7 mm
- board text removed: "GP10"
- board text removed: "GP16"
- board text removed: "GP18"
- board text removed: "GP19"
- board text removed: "GP20"
- board text removed: "GP21"

Commit message: some changes
Parts:
- removed G***: LOGO, logo:logo_Horizontal_small
- added J6: Camera2, Connector_FFC-FPC:Molex_54548-1071_1x10-1MP_P0.5mm_Horizontal, F.Cu at (175.5, 41.6)
- moved J2 84.4 mm to (176.5, 53.3), turned to -90 degrees
- moved J3 13.4 mm to (108.0, 40.6)
- moved J1 13.3 mm to (108.0, 52.6)
- moved U1 3.19 mm to (142.2, 47.0)
Connections:
- J3 pad 1: +3.3V -> 3.3V
- J3 pad 2: SCL_Cam1 -> SCL_Cam
- TP2 pad 1: +3.3V -> 3.3V
- TP4 pad 1: +3.3V -> 3.3V
- TP6 pad 1: +3.3V -> 3.3V
- U1 pad 10: DC_Cam2 -> DC_LED2
- U1 pad 11: unconnected-(U1-GPIO8-Pad11) -> VSYNC_Cam2
- U1 pad 12: unconnected-(U1-GPIO9-Pad12)_1 -> HREF_Cam2
- U1 pad 14: /GP10 -> DO_Cam1
- U1 pad 15: unconnected-(U1-GPIO11-Pad15)_1 -> PCLK_Cam2
- U1 pad 16: unconnected-(U1-GPIO12-Pad16) -> DO_Cam2
- U1 pad 17: CS_Cam1 -> CS_LED1
- U1 pad 19: RST_Cam1 -> RST_LED1
- U1 pad 20: DC_Cam1 -> DC_LED1
- U1 pad 21: /GP16 -> VSYNC_Cam1
- U1 pad 24: /GP18 -> PCLK_Cam1
- U1 pad 25: /GP19 -> HREF_Cam1
- U1 pad 26: /GP20 -> SDA_Cam1
- U1 pad 27: /GP21 -> SCL_Cam
- U1 pad 36: +3.3V -> 3.3V
- U1 pad 4: CLK_Cam -> CLK_LED
- U1 pad 5: DIN_Cam -> DIN_LED
- U1 pad 6: unconnected-(U1-GPIO4-Pad6)_1 -> SDA_Cam2
- U1 pad 7: CS_Cam2 -> CS_LED2
- U1 pad 9: RST_Cam2 -> RST_LED2
Routing:
- net DIN_LED: track 0.00 -> 79.6 mm, vias 0 -> 1
- net CLK_LED: track 0.00 -> 73.1 mm, vias 0 -> 1
- net 3.3V: track 0.00 -> 70.4 mm, vias 0 -> 1
- net SCL_Cam: track 0.00 -> 66.8 mm
- net VSYNC_Cam1: track 0.00 -> 65.0 mm, vias 0 -> 1
- net CLK_Cam: track 64.4 -> 0.00 mm
- net PCLK_Cam1: track 0.00 -> 59.0 mm
- net DIN_Cam: track 56.8 -> 0.00 mm
- net HREF_Cam1: track 0.00 -> 56.3 mm
- net SDA_Cam1: track 0.00 -> 52.9 mm
- net /GP16: track 51.3 -> 0.00 mm
- net CS_LED2: track 0.00 -> 50.5 mm
- net /GP18: track 48.6 -> 0.00 mm, vias 2 -> 0
- net RST_LED2: track 0.00 -> 46.9 mm, vias 0 -> 1
- net /GP19: track 44.7 -> 0.00 mm
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Other:
- board text removed: "3.3V"
- board text removed: "GND"
