File: Kicad Files/AR Glass/Glass_Old.kicad_sch (KiCad schematic)
At the start: 12 parts, among them J1 OLED1, J2 OLED2, J3 Camera1, J4 OLED1, J5 OLED2, U1 Pico

Commit message: work
Parts:
- removed J3: Camera1, Connector_FFC-FPC:Molex_54548-1071_1x10-1MP_P0.5mm_Horizontal, symbol Connector:Conn_01x08_Pin
- removed J4: OLED1, Connector_FFC-FPC:Molex_54548-1071_1x10-1MP_P0.5mm_Horizontal, symbol Connector:Conn_01x07_Pin
- removed J5: OLED2, Connector_FFC-FPC:Molex_54548-1071_1x10-1MP_P0.5mm_Horizontal, symbol Connector:Conn_01x07_Pin
- removed TP3: TestPoint, Connector_PinHeader_2.54mm:PinHeader_1x01_P2.54mm_Vertical, symbol Connector:TestPoint
- added TP7: TestPoint, Connector_PinHeader_2.54mm:PinHeader_1x01_P2.54mm_Vertical, symbol Connector:TestPoint
- added U2, U3: OLED Driver, Connector_PinHeader_2.54mm:PinHeader_1x07_P2.54mm_Vertical, symbol AR_Library:OLED Driver
- added U4: Camera, Connector_PinHeader_2.54mm:PinHeader_1x08_P2.54mm_Vertical, symbol AR_Library:Camera
- J1: value OLED1 -> Conn_01x07_Pin; footprint Connector_FFC-FPC:Molex_54548-1071_1x10-1MP_P0.5mm_Horizontal -> Connector_PinHeader_2.54mm:PinHeader_1x07_P2.54mm_Vertical
- J2: value OLED2 -> Conn_01x07_Pin; footprint Connector_FFC-FPC:Molex_54548-1071_1x10-1MP_P0.5mm_Horizontal -> Connector_PinHeader_2.54mm:PinHeader_1x07_P2.54mm_Vertical
- renumbered TP1 to TP2, TP2 to TP3
Connections:
- net 3.3V is gone; now on net +3.3V: J1.1 (Pin_1), J2.1 (Pin_1)
- net CLK_LED is gone; now on net GP2: J1.4 (Pin_4), J2.4 (Pin_4)
- net CS_LED1 is gone; now on net GP13: J1.5 (Pin_5)
- net CS_LED2 is gone; now on net GP5: J2.5 (Pin_5)
- net DC_LED1 is gone; now on net GP15: J1.6 (Pin_6)
- net DC_LED2 is gone; now on net GP7: J2.6 (Pin_6)
- net DIN_LED is gone; now on net GP3: J1.3 (Pin_3), J2.3 (Pin_3)
- net RST_LED1 is gone; now on net GP14: J1.7 (Pin_7)
- net RST_LED2 is gone; now on net GP6: J2.7 (Pin_7)
- net +3.3V: now also TP5.1, TP7.1, U2.1 (VCC), U3.1 (VCC), U4.1 (VCC); no longer TP4.1, TP6.1
- net GND: now also TP4.1, TP6.1, U2.2 (GND), U3.2 (GND), U4.8 (GND); no longer TP5.1
- net GP10: now also U4.7 (DO)
- net GP16: now also U4.4 (VSYNC)
- net GP18: now also U4.6 (PCLK)
- net GP19: now also U4.5 (HREF)
- net GP20: now also U4.3 (SDA)
- net GP21: now also U4.2 (SCL)
- net CLK_Cam renamed GP2
- net GP2: now also U2.4 (CLK), U3.4 (CLK)
- net CS_Cam1 renamed GP13
- net GP13: now also U2.5 (CS)
- net CS_Cam2 renamed GP5
- net GP5: now also U3.5 (CS)
- net DC_Cam1 renamed GP15
- net GP15: now also U2.6 (DC)
- net DC_Cam2 renamed GP7
- net GP7: now also U3.6 (DC)
- net DIN_Cam renamed GP3
- net GP3: now also U2.3 (DIN), U3.3 (DIN)
- net RST_Cam1 renamed GP14
- net GP14: now also U2.7 (RST)
- net RST_Cam2 renamed GP6
- net GP6: now also U3.7 (RST)
Other:
- moved on the sheet: J1, J2, TP2, TP3
