File: Kicad Files/EEG/Channel/Channel.kicad_pcb (KiCad board)
At the start: 2 copper layers, 74.9 x 20.3 mm, 29 parts, among them J1 Conn_01x02_Pin, J2 Conn_01x07_Pin, U1 INA823, U2 LF356N, U3 LF356N, U4 LF356N, U5 LF356N, U6 MCP4161

Commit message: Gerber generated
Parts:
- moved G*** 1.67 mm to (95.5, 78.0)
Changed lines of the file:
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@@
 			(outputformat 1)
 			(mirror no)
-			(drillshape 1)
+			(drillshape 0)
 			(scaleselection 1)
-			(outputdirectory "")
+			(outputdirectory "../Gerber_channel")
 		)
 	)
@@
 	(footprint "logo:logo_Horizontal_small"
 		(layer "B.Cu")
-		(at 93.98 77.47)
+		(at 95.55 78.04)
 		(property "Reference" "G***"
-			(at 0 0 360)
+			(at 0 0 0)
 			(layer "B.SilkS")
 			(hide yes)
@@
 		)
 		(property "Value" "LOGO"
-			(at 0.75 0 360)
+			(at 0.75 0 0)
 			(layer "B.SilkS")
 			(hide yes)
@@
 		)
 		(property "Footprint" "logo:logo_Horizontal_small"
-			(at 0 0 360)
+			(at 0 0 0)
 			(layer "B.Fab")
 			(hide yes)
@@
 		)
 		(property "Datasheet" ""
-			(at 0 0 360)
+			(at 0 0 0)
 			(layer "B.Fab")
 			(hide yes)
@@
 		)
 		(property "Description" ""
-			(at 0 0 360)
+			(at 0 0 0)
 			(layer "B.Fab")
 			(hide yes)

Commit message: AR revised
Parts:
- J2: moved to B.Cu
- turned J2 to 180 degrees
Routing:
- net GND: track 22.3 -> 31.7 mm, vias 6 -> 7
- net Vss: vias 3 -> 2
- net Vdd: vias 2 -> 3
- net Out: vias 0 -> 1
