File: Kicad Files/EEG Old/Mother/Mother.kicad_pcb (KiCad board)
At the start: 2 copper layers, 66 x 116.8 mm, 13 parts, among them J1 Conn_01x05_Pin, U1 Teensy4.1

Commit message: EEG Power Updated
Parts:
- added J2: Conn_01x02_Pin, Connector_PinHeader_1.27mm:PinHeader_1x02_P1.27mm_Vertical, F.Cu at (114.3, 157.5)
- moved G*** 2.00 mm to (104.1, 131.5)
Connections:
- U1 pad 47: unconnected-(U1-GND-Pad47) -> pwr_GND
- U1 pad 48: unconnected-(U1-VIN-Pad48) -> Vin
Routing:
- net GND: track 193.6 -> 96.6 mm
- net pwr_GND: track 0.00 -> 24.6 mm, vias 0 -> 2
- net Vin: track 0.00 -> 19.1 mm
- net CKL: track 340.1 -> 336.6 mm
- net Vss: track 369.8 -> 367.1 mm
- net Vdd: track 384.8 -> 382.6 mm
- net SDI: track 347.1 -> 344.9 mm
