File: Kicad Files/EEG kicad — no golden fingers/EEG2.kicad_pcb (KiCad board)
At the start: 2 copper layers, 120.7 x 64.8 mm, 273 parts, among them J1 Conn_02x20_Top_Bottom, J2 Conn_01x05_Pin, U1 INA823, U10 LF356M, U11 LF356M, U12 LF356M, U13 LF356M, U14 LF356M, U15 LF356M, U16 LF356M, U17 LF356M, U18 LF356M, U19 LF356M, U2 INA823, U20 LF356M, U21 LF356M, U22 LF356M, U23 LF356M, U24 LF356M, U25 LF356M, U26 AD5293, U27 AD5293, U28 AD5293, U29 AD5293, U3 INA823, U30 AD5293, U31 Teensy4.1, U32 AD5293, U33 AD5293, U34 AD5293, U35 AD5293, U36 AD5293, U37 LF356M, U38 LF356M, U39 LF356M, U4 INA823, U40 LF356M, U41 LF356M, U42 LF356M, U43 LF356M, U44 LF356M, U45 LF356M, U46 LF356M, U47 LF356M, U48 LF356M, U49 LF356M, U5 INA823, U50 LF356M, U51 LF356M, U52 LF356M, U53 LF356M, U54 LF356M, U55 LF356M, U56 LF356M, U57 INA823, U58 INA823, U59 INA823, U6 LF356M, U60 INA823, U61 INA823, U7 LF356M, U8 LF356M, U9 LF356M

Commit message: Working on EEG
Parts:
- removed C11, C16, C18, C19, C20, C38, C39, C4, C40, C41, C42, C43, C44, C45, C5, C61, C62, C63, C64, C65, C66, C67, C68, C69, C70, C71, C72, C73, C74, C75, C76, C77, C78, C79, C80, C9: 1uF, Capacitor_SMD:C_0805_2012Metric
- removed the C14 at (73.7, 76.9)
- removed the C17 at (73.7, 85.9)
- removed the C22 at (69.0, 40.0)
- removed C24, C26, C27, C28, C29, C30, C33, C34, C35, C46, C47, C48, C49, C50, C51, C52, C53, C54, C55, C56, C57, C58, C59, C60: 0.22uF, Capacitor_SMD:C_0603_1608Metric
- removed the C25 at (69.0, 47.5)
- removed the C3 at (69.2, 73.9)
- removed the C32 at (69.0, 65.1)
- removed the C37 at (78.1, 70.9)
- removed the C8 at (69.2, 88.9)
- removed J2: Conn_01x05_Pin, Connector_PinHeader_1.27mm:PinHeader_1x05_P1.27mm_Vertical
- removed R10, R111, R112, R113, R114, R115, R119, R12, R121, R123, R124, R125, R19, R20: 2.64k, Resistor_SMD:R_0603_1608Metric
- removed R100, R103, R106, R108, R110, R28, R31: 100, Resistor_SMD:R_0805_2012Metric
- removed R101, R104, R34, R35, R38, R39, R40, R53, R54, R55, R76, R77, R78, R79, R82, R91, R92, R93, R94, R95, R96, R97, R98: 10k, Resistor_SMD:R_0603_1608Metric
- removed R102, R105, R107, R109, R126, R127, R128, R129, R130, R29, R32, R4, R45, R46, R47, R48, R5, R50, R51, R80, R81, R83, R84, R85, R86, R87, R88, R89, R90, R99: 1k, Resistor_SMD:R_0402_1005Metric
- removed R116, R117, R118, R120, R122, R14, R15: 1.32k, Resistor_SMD:R_0805_2012Metric
- removed the R13 at (69.2, 103.8)
- removed the R18 at (81.0, 40.0)
- removed the R25 at (73.6, 103.8)
- removed the R26 at (90.7, 104.5)
- removed the R3 at (154.2, 76.2)
- removed the R33 at (81.0, 52.5)
- removed the R37 at (81.0, 62.6)
- removed the R43 at (93.6, 92.6)
- removed the R44 at (93.6, 94.6)
- removed the R52 at (85.1, 45.0)
- removed the R57 at (93.6, 110.5)
- removed R58, R59, R60, R63, R64, R65, R66, R67, R68, R69, R70, R71, R72, R73, R74, R75: 150k, Resistor_SMD:R_0402_1005Metric
- removed the R62 at (96.5, 98.5)
- removed the R8 at (77.0, 57.6)
- removed the U10 at (26.9, 65.3)
- removed the U11 at (26.9, 71.7)
- removed U12, U13, U14, U15, U18, U19, U20, U23, U24, U25, U37, U38, U39, U40, U41, U42, U43, U44, U45, U46, U47, U48, U49, U50, U51, U52, U53, U54, U55, U56: LF356M, LF356M:SOIC127P599X175-8N
- removed the U17 at (35.9, 52.4)
- removed the U22 at (35.9, 84.6)
- removed the U27 at (34.0, 98.6)
- removed U28, U29, U30, U32, U33, U34, U35, U36: AD5293, AD5293:AD5293
- removed the U3 at (156.4, 59.7)
- removed U4, U5, U57, U58, U59, U60, U61: INA823, Package_SO:VSSOP-8_3x3mm_P0.65mm
- added C14: 1uF, Capacitor_SMD:C_0805_2012Metric, F.Cu at (157.5, 85.1)
- added C14: 1uF, Capacitor_SMD:C_0805_2012Metric, F.Cu at (157.5, 59.2)
- added C14: 1uF, Capacitor_SMD:C_0805_2012Metric, F.Cu at (157.5, 72.4)
- added C17: 1uF, Capacitor_SMD:C_0805_2012Metric, F.Cu at (155.3, 66.4)
- added C17: 1uF, Capacitor_SMD:C_0805_2012Metric, F.Cu at (155.3, 79.1)
- added C17: 1uF, Capacitor_SMD:C_0805_2012Metric, F.Cu at (155.3, 53.2)
- added C22: 0.22uF, Capacitor_SMD:C_0603_1608Metric, F.Cu at (177.4, 78.0)
- added C22: 0.22uF, Capacitor_SMD:C_0603_1608Metric, F.Cu at (177.4, 52.1)
- added C22: 0.22uF, Capacitor_SMD:C_0603_1608Metric, F.Cu at (177.4, 65.3)
- added C22: 0.22uF, Capacitor_SMD:C_0603_1608Metric, F.Cu at (177.4, 39.4)
- added C25: 0.22uF, Capacitor_SMD:C_0603_1608Metric, F.Cu at (173.5, 78.0)
- added C25: 0.22uF, Capacitor_SMD:C_0603_1608Metric, F.Cu at (173.5, 39.4)
- added C25: 0.22uF, Capacitor_SMD:C_0603_1608Metric, F.Cu at (173.5, 52.1)
- added C25: 0.22uF, Capacitor_SMD:C_0603_1608Metric, F.Cu at (173.5, 65.3)
- added C3: 1uF, Capacitor_SMD:C_0805_2012Metric, F.Cu at (151.1, 66.4)
- added C3: 1uF, Capacitor_SMD:C_0805_2012Metric, F.Cu at (151.1, 79.1)
- added C3: 1uF, Capacitor_SMD:C_0805_2012Metric, F.Cu at (151.2, 53.2)
- added C32: 0.22uF, Capacitor_SMD:C_0603_1608Metric, F.Cu at (185.0, 57.1)
- added C32: 0.22uF, Capacitor_SMD:C_0603_1608Metric, F.Cu at (185.0, 70.4)
- added C32: 0.22uF, Capacitor_SMD:C_0603_1608Metric, F.Cu at (185.0, 83.1)
- added C32: 0.22uF, Capacitor_SMD:C_0603_1608Metric, F.Cu at (185.0, 44.5)
- added C37: 1uF, Capacitor_SMD:C_0805_2012Metric, F.Cu at (198.1, 41.9)
- added C37: 1uF, Capacitor_SMD:C_0805_2012Metric, F.Cu at (198.2, 54.6)
- added C37: 1uF, Capacitor_SMD:C_0805_2012Metric, F.Cu at (198.1, 67.8)
- added C37: 1uF, Capacitor_SMD:C_0805_2012Metric, F.Cu at (198.1, 80.5)
- added C8: 1uF, Capacitor_SMD:C_0805_2012Metric, F.Cu at (153.4, 59.2)
- added C8: 1uF, Capacitor_SMD:C_0805_2012Metric, F.Cu at (153.3, 85.1)
- added C8: 1uF, Capacitor_SMD:C_0805_2012Metric, F.Cu at (153.3, 72.4)
- added R13: 1.32k, Resistor_SMD:R_0805_2012Metric, F.Cu at (159.1, 79.1)
- added R13: 1.32k, Resistor_SMD:R_0805_2012Metric, F.Cu at (159.1, 53.2)
- added R13: 1.32k, Resistor_SMD:R_0805_2012Metric, F.Cu at (159.1, 66.4)
- added R18: 2.64k, Resistor_SMD:R_0603_1608Metric, F.Cu at (157.5, 69.0)
- added R18: 2.64k, Resistor_SMD:R_0603_1608Metric, F.Cu at (157.5, 55.8)
- added R18: 2.64k, Resistor_SMD:R_0603_1608Metric, F.Cu at (157.5, 81.7)
- added R25: 100, Resistor_SMD:R_0805_2012Metric, F.Cu at (170.2, 84.3)
- added R25: 100, Resistor_SMD:R_0805_2012Metric, F.Cu at (170.2, 58.4)
- added R25: 100, Resistor_SMD:R_0805_2012Metric, F.Cu at (170.2, 71.6)
- added R26: 1k, Resistor_SMD:R_0402_1005Metric, F.Cu at (170.2, 53.3)
- added R26: 1k, Resistor_SMD:R_0402_1005Metric, F.Cu at (170.2, 79.2)
- added R26: 1k, Resistor_SMD:R_0402_1005Metric, F.Cu at (170.2, 66.5)
- added R3: 1k, Resistor_SMD:R_0402_1005Metric, F.Cu at (147.4, 66.4)
- added R3: 1k, Resistor_SMD:R_0402_1005Metric, F.Cu at (147.4, 79.1)
- added R3: 1k, Resistor_SMD:R_0402_1005Metric, F.Cu at (147.4, 53.2)
- added R33: 10k, Resistor_SMD:R_0603_1608Metric, F.Cu at (173.5, 61.0)
- added R33: 10k, Resistor_SMD:R_0603_1608Metric, F.Cu at (173.5, 86.9)
- added R33: 10k, Resistor_SMD:R_0603_1608Metric, F.Cu at (173.5, 74.2)
- added R37: 10k, Resistor_SMD:R_0603_1608Metric, F.Cu at (177.4, 48.3)
- added R37: 10k, Resistor_SMD:R_0603_1608Metric, F.Cu at (177.4, 74.2)
- added R37: 10k, Resistor_SMD:R_0603_1608Metric, F.Cu at (177.4, 61.0)
- added R37: 10k, Resistor_SMD:R_0603_1608Metric, F.Cu at (177.4, 86.9)
- added R43: 1k, Resistor_SMD:R_0402_1005Metric, F.Cu at (180.9, 39.4)
- added R43: 1k, Resistor_SMD:R_0402_1005Metric, F.Cu at (180.9, 78.0)
- added R43: 1k, Resistor_SMD:R_0402_1005Metric, F.Cu at (180.9, 52.1)
- added R43: 1k, Resistor_SMD:R_0402_1005Metric, F.Cu at (180.9, 65.3)
- added R44: 1k, Resistor_SMD:R_0402_1005Metric, F.Cu at (180.9, 48.3)
- added R44: 1k, Resistor_SMD:R_0402_1005Metric, F.Cu at (180.9, 61.0)
- added R44: 1k, Resistor_SMD:R_0402_1005Metric, F.Cu at (180.9, 74.2)
- added R44: 1k, Resistor_SMD:R_0402_1005Metric, F.Cu at (180.9, 86.9)
- added R52: 10k, Resistor_SMD:R_0603_1608Metric, F.Cu at (185.0, 67.8)
- added R52: 10k, Resistor_SMD:R_0603_1608Metric, F.Cu at (185.0, 80.5)
- added R52: 10k, Resistor_SMD:R_0603_1608Metric, F.Cu at (185.0, 54.6)
- added R52: 10k, Resistor_SMD:R_0603_1608Metric, F.Cu at (185.0, 41.9)
- added R57: 150k, Resistor_SMD:R_0402_1005Metric, F.Cu at (198.2, 57.1)
- added R57: 150k, Resistor_SMD:R_0402_1005Metric, F.Cu at (198.1, 70.4)
- added R57: 150k, Resistor_SMD:R_0402_1005Metric, F.Cu at (198.1, 44.5)
- added R57: 150k, Resistor_SMD:R_0402_1005Metric, F.Cu at (198.1, 83.1)
- added R62: 150k, Resistor_SMD:R_0402_1005Metric, F.Cu at (204.6, 39.4)
- added R62: 150k, Resistor_SMD:R_0402_1005Metric, F.Cu at (204.6, 52.1)
- added R62: 150k, Resistor_SMD:R_0402_1005Metric, F.Cu at (204.6, 65.3)
- added R62: 150k, Resistor_SMD:R_0402_1005Metric, F.Cu at (204.6, 78.0)
- added R8: 2.64k, Resistor_SMD:R_0603_1608Metric, F.Cu at (153.4, 55.8)
- added R8: 2.64k, Resistor_SMD:R_0603_1608Metric, F.Cu at (153.3, 69.0)
- added R8: 2.64k, Resistor_SMD:R_0603_1608Metric, F.Cu at (153.3, 81.7)
- added U10: LF356M, LF356M:SOIC127P599X175-8N, F.Cu at (165.1, 66.4)
- added U10: LF356M, LF356M:SOIC127P599X175-8N, F.Cu at (165.1, 53.2)
- added U10: LF356M, LF356M:SOIC127P599X175-8N, F.Cu at (165.1, 79.1)
- added U11: LF356M, LF356M:SOIC127P599X175-8N, F.Cu at (165.1, 85.6)
- added U11: LF356M, LF356M:SOIC127P599X175-8N, F.Cu at (165.1, 72.9)
- added U11: LF356M, LF356M:SOIC127P599X175-8N, F.Cu at (165.1, 59.7)
- added U17: LF356M, LF356M:SOIC127P599X175-8N, F.Cu at (176.5, 81.8)
- added U17: LF356M, LF356M:SOIC127P599X175-8N, F.Cu at (176.6, 55.9)
- added U17: LF356M, LF356M:SOIC127P599X175-8N, F.Cu at (176.5, 43.2)
- added U17: LF356M, LF356M:SOIC127P599X175-8N, F.Cu at (176.5, 69.1)
- added U22: LF356M, LF356M:SOIC127P599X175-8N, F.Cu at (191.8, 55.9)
- added U22: LF356M, LF356M:SOIC127P599X175-8N, F.Cu at (191.8, 43.2)
- added U22: LF356M, LF356M:SOIC127P599X175-8N, F.Cu at (191.8, 81.8)
- added U22: LF356M, LF356M:SOIC127P599X175-8N, F.Cu at (191.8, 69.1)
- added U27: AD5293, AD5293:AD5293, F.Cu at (204.5, 69.1)
- added U27: AD5293, AD5293:AD5293, F.Cu at (204.5, 55.9)
- added U27: AD5293, AD5293:AD5293, F.Cu at (204.5, 43.2)
- added U27: AD5293, AD5293:AD5293, F.Cu at (204.5, 81.8)
- added U3: INA823, Package_SO:VSSOP-8_3x3mm_P0.65mm, F.Cu at (147.3, 70.2)
- added U3: INA823, Package_SO:VSSOP-8_3x3mm_P0.65mm, F.Cu at (147.3, 57.0)
- added U3: INA823, Package_SO:VSSOP-8_3x3mm_P0.65mm, F.Cu at (147.3, 83.0)
- moved U8 138.7 mm to (165.1, 40.5)
- moved U9 138.7 mm to (165.1, 47.0)
- moved R61 128.7 mm to (204.6, 26.7)
- moved R23 111.2 mm to (170.2, 45.7), turned to 90 degrees
- moved R11 108.2 mm to (159.1, 40.5)
- moved R24 100.7 mm to (170.2, 40.6)
- moved C7 92.9 mm to (153.3, 46.5), turned to 180 degrees
- moved R30 92.5 mm to (173.5, 48.3)
- moved C15 90.6 mm to (155.3, 40.5)
- moved C2 87.3 mm to (151.1, 40.5)
- moved C12 87.3 mm to (157.5, 46.5), turned to 180 degrees
- moved R7 77.2 mm to (153.3, 43.1), turned to 180 degrees
- moved R17 76.6 mm to (157.5, 43.1), turned to 180 degrees
- moved R2 34.4 mm to (147.4, 40.5)
- moved U2 14.0 mm to (147.3, 44.3)
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Connections:
- C12 pad 1: Net-(U8--) -> Net-(U6--)
- C12 pad 2: Net-(C12-Pad2) -> Net-(C10-Pad2)
- C15 pad 1: Net-(C15-Pad1) -> Net-(C1-Pad2)
- C15 pad 2: Net-(U9-+) -> Net-(U7-+)
- C2 pad 1: Net-(C2-Pad1) -> Net-(C1-Pad1)
- C2 pad 2: Net-(C15-Pad1) -> Net-(C1-Pad2)
- C7 pad 1: Net-(U8--) -> Net-(U6--)
- C7 pad 2: Net-(C12-Pad2) -> Net-(C10-Pad2)
- R11 pad 1: Net-(C15-Pad1) -> Net-(C1-Pad2)
- R11 pad 2: Net-(U8--) -> Net-(U6--)
- R17 pad 1: Net-(U9-+) -> Net-(U7-+)
- R17 pad 2: Net-(C12-Pad2) -> Net-(C10-Pad2)
- R2 pad 1: Net-(R2-Pad1) -> Net-(R1-Pad1)
- R2 pad 2: Net-(R2-Pad2) -> Net-(R1-Pad2)
- R23 pad 1: Net-(U9--) -> Net-(U7--)
- R23 pad 2: Net-(U8-+) -> Net-(U6-+)
- R24 pad 1: Net-(U8-+) -> Net-(U6-+)
- R30 pad 1: Net-(U9--) -> Net-(U7--)
- R30 pad 2: Net-(C25-Pad2) -> Net-(C23-Pad2)
- R7 pad 1: Net-(C12-Pad2) -> Net-(C10-Pad2)
- R7 pad 2: Net-(C2-Pad1) -> Net-(C1-Pad1)
- U2 pad 1: Net-(R2-Pad1) -> Net-(R1-Pad1)
- U2 pad 3: Electrode2 -> Electrode1
- U2 pad 6: Net-(C2-Pad1) -> Net-(C1-Pad1)
- U2 pad 8: Net-(R2-Pad2) -> Net-(R1-Pad2)
- U8 pad 1: unconnected-(U8-NULL-Pad1) -> unconnected-(U6-NULL-Pad1)
- U8 pad 2: Net-(U8--) -> Net-(U6--)
- U8 pad 3: Net-(U8-+) -> Net-(U6-+)
- U8 pad 5: unconnected-(U8-NULL-Pad5) -> unconnected-(U6-NULL-Pad5)
- U8 pad 6: Net-(U8--) -> Net-(U6--)
- U8 pad 8: unconnected-(U8-NC-Pad8) -> unconnected-(U6-NC-Pad8)
- U9 pad 1: unconnected-(U9-NULL-Pad1) -> unconnected-(U7-NULL-Pad1)
- U9 pad 2: Net-(U9--) -> Net-(U7--)
- U9 pad 3: Net-(U9-+) -> Net-(U7-+)
- U9 pad 5: unconnected-(U9-NULL-Pad5) -> unconnected-(U7-NULL-Pad5)
- U9 pad 6: Net-(U9--) -> Net-(U7--)
- U9 pad 8: unconnected-(U9-NC-Pad8) -> unconnected-(U7-NC-Pad8)
Routing:
- net Net-(U6--): track 0.00 -> 20.7 mm, vias 0 -> 2
- net Net-(C23-Pad1): track 0.00 -> 17.3 mm
- net Net-(U6-+): track 0.00 -> 12.4 mm
- net Net-(C23-Pad2): track 0.00 -> 11.8 mm
- net Net-(U7--): track 0.00 -> 11.6 mm
- net Net-(U16--): track 0.00 -> 10.6 mm
- net Net-(C10-Pad2): track 0.00 -> 10.1 mm
- net Net-(U7-+): track 0.00 -> 9.98 mm
- net Net-(C1-Pad2): track 0.00 -> 7.54 mm
- net Net-(C1-Pad1): track 0.00 -> 7.26 mm
- net Net-(U21-+): track 0.00 -> 6.37 mm
- net Electrode Output 1: track 0.00 -> 6.03 mm
- net Net-(C36-Pad1): track 0.00 -> 5.62 mm
- net Net-(U16-+): track 0.00 -> 5.20 mm
- net Net-(R1-Pad1): track 0.00 -> 3.53 mm
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Other:
- board size 120.7 x 64.8 mm -> 109.2 x 64.8 mm

Commit message: Working on EEG
Parts:
- removed the C22 at (177.4, 78.0)
- removed the C22 at (177.4, 52.1)
- removed the C22 at (177.4, 65.3)
- removed the C25 at (173.5, 78.0)
- removed the C25 at (173.5, 52.1)
- removed the C25 at (173.5, 65.3)
- removed the C32 at (185.0, 57.1)
- removed the C32 at (185.0, 70.4)
- removed the C32 at (185.0, 83.1)
- removed the C37 at (198.2, 54.6)
- removed the C37 at (198.1, 67.8)
- removed the C37 at (198.1, 80.5)
- removed the R25 at (170.2, 84.3)
- removed the R25 at (170.2, 71.6)
- removed the R26 at (170.2, 79.2)
- removed the R26 at (170.2, 66.5)
- removed the R33 at (173.5, 61.0)
- removed the R33 at (173.5, 86.9)
- removed the R33 at (173.5, 74.2)
- removed the R37 at (177.4, 74.2)
- removed the R37 at (177.4, 61.0)
- removed the R37 at (177.4, 86.9)
- removed the R43 at (180.9, 78.0)
- removed the R43 at (180.9, 52.1)
- removed the R43 at (180.9, 65.3)
- removed the R44 at (180.9, 61.0)
- removed the R44 at (180.9, 74.2)
- removed the R44 at (180.9, 86.9)
- removed the R52 at (185.0, 67.8)
- removed the R52 at (185.0, 80.5)
- removed the R52 at (185.0, 54.6)
- removed the R57 at (198.2, 57.1)
- removed the R57 at (198.1, 70.4)
- removed the R57 at (198.1, 83.1)
- removed the R62 at (204.6, 52.1)
- removed the R62 at (204.6, 65.3)
- removed the R62 at (204.6, 78.0)
- removed the U17 at (176.5, 81.8)
- removed the U17 at (176.6, 55.9)
- removed the U17 at (176.5, 69.1)
- removed the U22 at (191.8, 55.9)
- removed the U22 at (191.8, 81.8)
- removed the U22 at (191.8, 69.1)
- removed the U27 at (204.5, 69.1)
- removed the U27 at (204.5, 55.9)
- removed the U27 at (204.5, 81.8)
- added C24: 0.22uF, Capacitor_SMD:C_0603_1608Metric, F.Cu at (177.3, 52.1)
- added C26: 0.22uF, Capacitor_SMD:C_0603_1608Metric, F.Cu at (177.4, 66.0)
- added C27: 0.22uF, Capacitor_SMD:C_0603_1608Metric, F.Cu at (173.4, 52.1)
- added C28: 0.22uF, Capacitor_SMD:C_0603_1608Metric, F.Cu at (177.4, 78.7)
- added C29: 0.22uF, Capacitor_SMD:C_0603_1608Metric, F.Cu at (173.5, 66.0)
- added C30: 0.22uF, Capacitor_SMD:C_0603_1608Metric, F.Cu at (173.5, 78.7)
- added C33: 0.22uF, Capacitor_SMD:C_0603_1608Metric, F.Cu at (184.9, 57.1)
- added C34: 0.22uF, Capacitor_SMD:C_0603_1608Metric, F.Cu at (185.0, 71.1)
- added C35: 0.22uF, Capacitor_SMD:C_0603_1608Metric, F.Cu at (185.0, 83.8)
- added C38: 1uF, Capacitor_SMD:C_0805_2012Metric, F.Cu at (198.1, 54.6)
- added C39: 1uF, Capacitor_SMD:C_0805_2012Metric, F.Cu at (198.1, 68.6)
- added C40: 1uF, Capacitor_SMD:C_0805_2012Metric, F.Cu at (198.1, 81.3)
- added C41: 1uF, Capacitor_SMD:C_0805_2012Metric, F.Cu at (198.1, 93.2)
- added C42: 1uF, Capacitor_SMD:C_0805_2012Metric, F.Cu at (198.2, 106.2)
- added C43: 1uF, Capacitor_SMD:C_0805_2012Metric, F.Cu at (198.3, 119.3)
- added C44: 1uF, Capacitor_SMD:C_0805_2012Metric, F.Cu at (198.3, 132.4)
- added C45: 1uF, Capacitor_SMD:C_0805_2012Metric, F.Cu at (198.4, 145.5)
- added C46: 0.22uF, Capacitor_SMD:C_0603_1608Metric, F.Cu at (185.0, 95.8)
- added C47: 0.22uF, Capacitor_SMD:C_0603_1608Metric, F.Cu at (185.1, 108.7)
- added C48: 0.22uF, Capacitor_SMD:C_0603_1608Metric, F.Cu at (185.1, 121.8)
- added C49: 0.22uF, Capacitor_SMD:C_0603_1608Metric, F.Cu at (185.2, 134.9)
- added C50: 0.22uF, Capacitor_SMD:C_0603_1608Metric, F.Cu at (185.2, 148.1)
- added C51: 0.22uF, Capacitor_SMD:C_0603_1608Metric, F.Cu at (173.5, 90.7)
- added C52: 0.22uF, Capacitor_SMD:C_0603_1608Metric, F.Cu at (173.6, 103.6)
- added C53: 0.22uF, Capacitor_SMD:C_0603_1608Metric, F.Cu at (177.4, 90.7)
- added C54: 0.22uF, Capacitor_SMD:C_0603_1608Metric, F.Cu at (173.6, 116.8)
- added C55: 0.22uF, Capacitor_SMD:C_0603_1608Metric, F.Cu at (177.5, 103.6)
- added C56: 0.22uF, Capacitor_SMD:C_0603_1608Metric, F.Cu at (173.7, 129.9)
- added C57: 0.22uF, Capacitor_SMD:C_0603_1608Metric, F.Cu at (177.5, 116.8)
- added C58: 0.22uF, Capacitor_SMD:C_0603_1608Metric, F.Cu at (173.7, 143.0)
- added C59: 0.22uF, Capacitor_SMD:C_0603_1608Metric, F.Cu at (177.6, 129.9)
- added C60: 0.22uF, Capacitor_SMD:C_0603_1608Metric, F.Cu at (177.6, 143.0)
- added C61: 1uF, Capacitor_SMD:C_0805_2012Metric, F.Cu at (155.3, 92.0)
- added C62: 1uF, Capacitor_SMD:C_0805_2012Metric, F.Cu at (155.4, 104.9)
- added C63: 1uF, Capacitor_SMD:C_0805_2012Metric, F.Cu at (153.4, 97.9)
- added C64: 1uF, Capacitor_SMD:C_0805_2012Metric, F.Cu at (155.4, 118.0)
- added C65: 1uF, Capacitor_SMD:C_0805_2012Metric, F.Cu at (153.4, 110.9)
- added C66: 1uF, Capacitor_SMD:C_0805_2012Metric, F.Cu at (155.5, 131.1)
- added C67: 1uF, Capacitor_SMD:C_0805_2012Metric, F.Cu at (153.5, 124.0)
- added C68: 1uF, Capacitor_SMD:C_0805_2012Metric, F.Cu at (155.5, 144.3)
- added C69: 1uF, Capacitor_SMD:C_0805_2012Metric, F.Cu at (153.5, 137.1)
- added C70: 1uF, Capacitor_SMD:C_0805_2012Metric, F.Cu at (157.5, 97.9)
- added C71: 1uF, Capacitor_SMD:C_0805_2012Metric, F.Cu at (153.6, 150.2)
- added C72: 1uF, Capacitor_SMD:C_0805_2012Metric, F.Cu at (157.6, 110.9)
- added C73: 1uF, Capacitor_SMD:C_0805_2012Metric, F.Cu at (157.6, 124.0)
- added C74: 1uF, Capacitor_SMD:C_0805_2012Metric, F.Cu at (157.7, 137.1)
- added C75: 1uF, Capacitor_SMD:C_0805_2012Metric, F.Cu at (157.7, 150.2)
- added C76: 1uF, Capacitor_SMD:C_0805_2012Metric, F.Cu at (151.2, 92.0)
- added C77: 1uF, Capacitor_SMD:C_0805_2012Metric, F.Cu at (151.2, 104.9)
- added C78: 1uF, Capacitor_SMD:C_0805_2012Metric, F.Cu at (151.3, 118.0)
- added C79: 1uF, Capacitor_SMD:C_0805_2012Metric, F.Cu at (151.3, 131.1)
- added C80: 1uF, Capacitor_SMD:C_0805_2012Metric, F.Cu at (151.4, 144.3)
- added J2: Conn_01x05_Pin, Connector_PinHeader_1.27mm:PinHeader_1x05_P1.27mm_Vertical, F.Cu at (214.6, 90.2)
- added R100: 100, Resistor_SMD:R_0805_2012Metric, F.Cu at (170.2, 97.0)
- added R101: 10k, Resistor_SMD:R_0603_1608Metric, F.Cu at (173.6, 138.8)
- added R102: 1k, Resistor_SMD:R_0402_1005Metric, F.Cu at (170.3, 104.9)
- added R103: 100, Resistor_SMD:R_0805_2012Metric, F.Cu at (170.3, 110.0)
- added R104: 10k, Resistor_SMD:R_0603_1608Metric, F.Cu at (173.7, 151.9)
- added R105: 1k, Resistor_SMD:R_0402_1005Metric, F.Cu at (170.3, 123.1)
- added R106: 100, Resistor_SMD:R_0805_2012Metric, F.Cu at (170.3, 118.0)
- added R107: 1k, Resistor_SMD:R_0402_1005Metric, F.Cu at (170.4, 136.2)
- added R108: 100, Resistor_SMD:R_0805_2012Metric, F.Cu at (170.4, 131.1)
- added R109: 1k, Resistor_SMD:R_0402_1005Metric, F.Cu at (170.4, 149.3)
- added R110: 100, Resistor_SMD:R_0805_2012Metric, F.Cu at (170.4, 144.3)
- added R111: 2.64k, Resistor_SMD:R_0603_1608Metric, F.Cu at (157.5, 94.5)
- added R112: 2.64k, Resistor_SMD:R_0603_1608Metric, F.Cu at (157.6, 107.5)
- added R113: 2.64k, Resistor_SMD:R_0603_1608Metric, F.Cu at (157.6, 120.6)
- added R114: 2.64k, Resistor_SMD:R_0603_1608Metric, F.Cu at (157.7, 133.7)
- added R115: 2.64k, Resistor_SMD:R_0603_1608Metric, F.Cu at (157.7, 146.8)
- added R116: 1.32k, Resistor_SMD:R_0805_2012Metric, F.Cu at (159.1, 92.0)
- added R117: 1.32k, Resistor_SMD:R_0805_2012Metric, F.Cu at (159.2, 104.9)
- added R118: 1.32k, Resistor_SMD:R_0805_2012Metric, F.Cu at (159.2, 118.0)
- added R119: 2.64k, Resistor_SMD:R_0603_1608Metric, F.Cu at (153.4, 94.5)
- added R120: 1.32k, Resistor_SMD:R_0805_2012Metric, F.Cu at (159.3, 131.1)
- added R121: 2.64k, Resistor_SMD:R_0603_1608Metric, F.Cu at (153.4, 107.5)
- added R122: 1.32k, Resistor_SMD:R_0805_2012Metric, F.Cu at (159.3, 144.3)
- added R123: 2.64k, Resistor_SMD:R_0603_1608Metric, F.Cu at (153.5, 120.6)
- added R124: 2.64k, Resistor_SMD:R_0603_1608Metric, F.Cu at (153.5, 133.7)
- added R125: 2.64k, Resistor_SMD:R_0603_1608Metric, F.Cu at (153.6, 146.8)
- added R126: 1k, Resistor_SMD:R_0402_1005Metric, F.Cu at (147.4, 92.0)
- added R127: 1k, Resistor_SMD:R_0402_1005Metric, F.Cu at (147.5, 104.9)
- added R128: 1k, Resistor_SMD:R_0402_1005Metric, F.Cu at (147.5, 118.0)
- added R129: 1k, Resistor_SMD:R_0402_1005Metric, F.Cu at (147.6, 131.1)
- added R130: 1k, Resistor_SMD:R_0402_1005Metric, F.Cu at (147.6, 144.3)
- added R28: 100, Resistor_SMD:R_0805_2012Metric, F.Cu at (170.2, 72.4)
- added R29: 1k, Resistor_SMD:R_0402_1005Metric, F.Cu at (170.2, 67.3)
- added R31: 100, Resistor_SMD:R_0805_2012Metric, F.Cu at (170.2, 85.1)
- added R32: 1k, Resistor_SMD:R_0402_1005Metric, F.Cu at (170.2, 80.0)
- added R33: 10k, Resistor_SMD:R_0603_1608Metric, F.Cu at (173.4, 61.0)
- added R34: 10k, Resistor_SMD:R_0603_1608Metric, F.Cu at (173.5, 74.9)
- added R35: 10k, Resistor_SMD:R_0603_1608Metric, F.Cu at (173.5, 87.6)
- added R38: 10k, Resistor_SMD:R_0603_1608Metric, F.Cu at (177.3, 61.0)
- added R39: 10k, Resistor_SMD:R_0603_1608Metric, F.Cu at (177.4, 74.9)
- added R40: 10k, Resistor_SMD:R_0603_1608Metric, F.Cu at (177.4, 87.6)
- added R45: 1k, Resistor_SMD:R_0402_1005Metric, F.Cu at (180.8, 52.1)
- added R46: 1k, Resistor_SMD:R_0402_1005Metric, F.Cu at (180.8, 61.0)
- added R47: 1k, Resistor_SMD:R_0402_1005Metric, F.Cu at (180.9, 66.0)
- added R48: 1k, Resistor_SMD:R_0402_1005Metric, F.Cu at (180.9, 74.9)
- added R50: 1k, Resistor_SMD:R_0402_1005Metric, F.Cu at (180.9, 78.7)
- added R51: 1k, Resistor_SMD:R_0402_1005Metric, F.Cu at (180.9, 87.6)
- added R53: 10k, Resistor_SMD:R_0603_1608Metric, F.Cu at (184.9, 54.6)
- added R54: 10k, Resistor_SMD:R_0603_1608Metric, F.Cu at (185.0, 68.6)
- added R55: 10k, Resistor_SMD:R_0603_1608Metric, F.Cu at (185.0, 81.3)
- added R58: 150k, Resistor_SMD:R_0402_1005Metric, F.Cu at (198.1, 57.1)
- added R59: 150k, Resistor_SMD:R_0402_1005Metric, F.Cu at (198.1, 71.1)
- added R60: 150k, Resistor_SMD:R_0402_1005Metric, F.Cu at (198.1, 83.8)
- added R63: 150k, Resistor_SMD:R_0402_1005Metric, F.Cu at (204.5, 52.1)
- added R64: 150k, Resistor_SMD:R_0402_1005Metric, F.Cu at (204.6, 66.0)
- added R65: 150k, Resistor_SMD:R_0402_1005Metric, F.Cu at (204.6, 78.7)
- added R66: 150k, Resistor_SMD:R_0402_1005Metric, F.Cu at (204.6, 90.7)
- added R67: 150k, Resistor_SMD:R_0402_1005Metric, F.Cu at (204.7, 103.6)
- added R68: 150k, Resistor_SMD:R_0402_1005Metric, F.Cu at (204.7, 116.8)
- added R69: 150k, Resistor_SMD:R_0402_1005Metric, F.Cu at (204.8, 129.9)
- added R70: 150k, Resistor_SMD:R_0402_1005Metric, F.Cu at (204.8, 143.0)
- added R71: 150k, Resistor_SMD:R_0402_1005Metric, F.Cu at (198.1, 95.8)
- added R72: 150k, Resistor_SMD:R_0402_1005Metric, F.Cu at (198.2, 108.7)
- added R73: 150k, Resistor_SMD:R_0402_1005Metric, F.Cu at (198.3, 121.8)
- added R74: 150k, Resistor_SMD:R_0402_1005Metric, F.Cu at (198.3, 134.9)
- added R75: 150k, Resistor_SMD:R_0402_1005Metric, F.Cu at (198.4, 148.1)
- added R76: 10k, Resistor_SMD:R_0603_1608Metric, F.Cu at (185.0, 93.2)
- added R77: 10k, Resistor_SMD:R_0603_1608Metric, F.Cu at (185.1, 106.2)
- added R78: 10k, Resistor_SMD:R_0603_1608Metric, F.Cu at (185.1, 119.3)
- added R79: 10k, Resistor_SMD:R_0603_1608Metric, F.Cu at (185.2, 132.4)
- added R80: 1k, Resistor_SMD:R_0402_1005Metric, F.Cu at (180.9, 99.6)
- added R81: 1k, Resistor_SMD:R_0402_1005Metric, F.Cu at (180.9, 90.7)
- added R82: 10k, Resistor_SMD:R_0603_1608Metric, F.Cu at (185.2, 145.5)
- added R83: 1k, Resistor_SMD:R_0402_1005Metric, F.Cu at (181.0, 112.5)
- added R84: 1k, Resistor_SMD:R_0402_1005Metric, F.Cu at (181.0, 103.6)
- added R85: 1k, Resistor_SMD:R_0402_1005Metric, F.Cu at (181.1, 125.7)
- added R86: 1k, Resistor_SMD:R_0402_1005Metric, F.Cu at (181.1, 116.8)
- added R87: 1k, Resistor_SMD:R_0402_1005Metric, F.Cu at (181.1, 138.8)
- added R88: 1k, Resistor_SMD:R_0402_1005Metric, F.Cu at (181.1, 129.9)
- added R89: 1k, Resistor_SMD:R_0402_1005Metric, F.Cu at (181.1, 151.9)
- added R90: 1k, Resistor_SMD:R_0402_1005Metric, F.Cu at (181.1, 143.0)
- added R91: 10k, Resistor_SMD:R_0603_1608Metric, F.Cu at (177.4, 99.6)
- added R92: 10k, Resistor_SMD:R_0603_1608Metric, F.Cu at (177.5, 112.5)
- added R93: 10k, Resistor_SMD:R_0603_1608Metric, F.Cu at (177.5, 125.7)
- added R94: 10k, Resistor_SMD:R_0603_1608Metric, F.Cu at (177.6, 138.8)
- added R95: 10k, Resistor_SMD:R_0603_1608Metric, F.Cu at (177.6, 151.9)
- added R96: 10k, Resistor_SMD:R_0603_1608Metric, F.Cu at (173.5, 99.6)
- added R97: 10k, Resistor_SMD:R_0603_1608Metric, F.Cu at (173.5, 112.5)
- added R98: 10k, Resistor_SMD:R_0603_1608Metric, F.Cu at (173.6, 125.7)
- added R99: 1k, Resistor_SMD:R_0402_1005Metric, F.Cu at (170.2, 92.0)
- added U18: LF356M, LF356M:SOIC127P599X175-8N, F.Cu at (176.5, 55.9)
- added U19: LF356M, LF356M:SOIC127P599X175-8N, F.Cu at (176.5, 69.8)
- added U20: LF356M, LF356M:SOIC127P599X175-8N, F.Cu at (176.5, 82.5)
- added U23: LF356M, LF356M:SOIC127P599X175-8N, F.Cu at (191.7, 55.9)
- added U24: LF356M, LF356M:SOIC127P599X175-8N, F.Cu at (191.8, 69.8)
- added U25: LF356M, LF356M:SOIC127P599X175-8N, F.Cu at (191.8, 82.5)
- added U28: AD5293, AD5293:AD5293, F.Cu at (204.4, 55.9)
- added U29: AD5293, AD5293:AD5293, F.Cu at (204.5, 69.8)
- added U30: AD5293, AD5293:AD5293, F.Cu at (204.5, 82.5)
- added U32: AD5293, AD5293:AD5293, F.Cu at (204.5, 94.5)
- added U33: AD5293, AD5293:AD5293, F.Cu at (204.6, 107.5)
- added U34: AD5293, AD5293:AD5293, F.Cu at (204.6, 120.6)
- added U35: AD5293, AD5293:AD5293, F.Cu at (204.7, 133.7)
- added U36: AD5293, AD5293:AD5293, F.Cu at (204.7, 146.8)
- added U37: LF356M, LF356M:SOIC127P599X175-8N, F.Cu at (191.8, 94.5)
- added U38: LF356M, LF356M:SOIC127P599X175-8N, F.Cu at (191.9, 107.5)
- added U39: LF356M, LF356M:SOIC127P599X175-8N, F.Cu at (191.9, 120.6)
- added U40: LF356M, LF356M:SOIC127P599X175-8N, F.Cu at (192.0, 133.7)
- added U41: LF356M, LF356M:SOIC127P599X175-8N, F.Cu at (192.0, 146.8)
- added U42: LF356M, LF356M:SOIC127P599X175-8N, F.Cu at (176.6, 94.5)
- added U43: LF356M, LF356M:SOIC127P599X175-8N, F.Cu at (176.6, 107.5)
- added U44: LF356M, LF356M:SOIC127P599X175-8N, F.Cu at (176.7, 120.6)
- added U45: LF356M, LF356M:SOIC127P599X175-8N, F.Cu at (176.7, 133.7)
- added U46: LF356M, LF356M:SOIC127P599X175-8N, F.Cu at (176.8, 146.8)
- added U47: LF356M, LF356M:SOIC127P599X175-8N, F.Cu at (165.1, 98.4)
- added U48: LF356M, LF356M:SOIC127P599X175-8N, F.Cu at (165.1, 92.0)
- added U49: LF356M, LF356M:SOIC127P599X175-8N, F.Cu at (165.2, 111.4)
- added U50: LF356M, LF356M:SOIC127P599X175-8N, F.Cu at (165.2, 104.9)
- added U51: LF356M, LF356M:SOIC127P599X175-8N, F.Cu at (165.2, 124.5)
- added U52: LF356M, LF356M:SOIC127P599X175-8N, F.Cu at (165.2, 118.0)
- added U53: LF356M, LF356M:SOIC127P599X175-8N, F.Cu at (165.3, 137.6)
- added U54: LF356M, LF356M:SOIC127P599X175-8N, F.Cu at (165.3, 131.1)
- added U55: LF356M, LF356M:SOIC127P599X175-8N, F.Cu at (165.3, 150.7)
- added U56: LF356M, LF356M:SOIC127P599X175-8N, F.Cu at (165.3, 144.3)
- added U57: INA823, Package_SO:VSSOP-8_3x3mm_P0.65mm, F.Cu at (147.3, 95.8)
- added U58: INA823, Package_SO:VSSOP-8_3x3mm_P0.65mm, F.Cu at (147.4, 108.7)
- added U59: INA823, Package_SO:VSSOP-8_3x3mm_P0.65mm, F.Cu at (147.3, 121.9)
- added U60: INA823, Package_SO:VSSOP-8_3x3mm_P0.65mm, F.Cu at (147.5, 134.9)
- added U61: INA823, Package_SO:VSSOP-8_3x3mm_P0.65mm, F.Cu at (147.6, 148.1)
- moved J1 34.3 mm to (133.3, 90.9)
- renumbered C8 to C11, C14 to C16, C14 to C18, C17 to C19, C17 to C20, C3 to C4, C3 to C5, C8 to C9, R8 to R10, R8 to R12, R13 to R14, R13 to R15, R18 to R19, R18 to R20, R3 to R4, R3 to R5, U10 to U12, U11 to U13, U10 to U14, U11 to U15, U3 to U4, U3 to U5
Connections:
- C11 pad 1: Net-(U6--) -> Net-(U14--)
- C11 pad 2: Net-(C10-Pad2) -> Net-(C11-Pad2)
- C12 pad 1: Net-(U6--) -> Net-(U8--)
- C12 pad 2: Net-(C10-Pad2) -> Net-(C12-Pad2)
- C14 pad 1: Net-(U6--) -> Net-(U10--)
- C14 pad 2: Net-(C10-Pad2) -> Net-(C14-Pad2)
- C15 pad 1: Net-(C1-Pad2) -> Net-(C15-Pad1)
- C15 pad 2: Net-(U7-+) -> Net-(U9-+)
- C16 pad 1: Net-(U6--) -> Net-(U12--)
- C16 pad 2: Net-(C10-Pad2) -> Net-(C16-Pad2)
- C17 pad 1: Net-(C1-Pad2) -> Net-(C17-Pad1)
- C17 pad 2: Net-(U7-+) -> Net-(U11-+)
- C18 pad 1: Net-(U6--) -> Net-(U14--)
- C18 pad 2: Net-(C10-Pad2) -> Net-(C11-Pad2)
- C19 pad 1: Net-(C1-Pad2) -> Net-(C19-Pad1)
- C19 pad 2: Net-(U7-+) -> Net-(U13-+)
- C2 pad 1: Net-(C1-Pad1) -> Net-(C2-Pad1)
- C2 pad 2: Net-(C1-Pad2) -> Net-(C15-Pad1)
- C20 pad 1: Net-(C1-Pad2) -> Net-(C20-Pad1)
- C20 pad 2: Net-(U7-+) -> Net-(U15-+)
- C22 pad 1: Net-(U16-+) -> Net-(U17-+)
- C25 pad 1: Net-(C23-Pad1) -> Net-(C25-Pad1)
- C25 pad 2: Net-(C23-Pad2) -> Net-(C25-Pad2)
- C3 pad 1: Net-(C1-Pad1) -> Net-(C3-Pad1)
- C3 pad 2: Net-(C1-Pad2) -> Net-(C17-Pad1)
- C32 pad 1: Net-(U21-+) -> Net-(U22-+)
- C37 pad 1: Net-(C36-Pad1) -> Net-(C37-Pad1)
- C37 pad 2: Electrode Output 1 -> Electrode Output 2
- C4 pad 1: Net-(C1-Pad1) -> Net-(C4-Pad1)
- C4 pad 2: Net-(C1-Pad2) -> Net-(C19-Pad1)
- C5 pad 1: Net-(C1-Pad1) -> Net-(C5-Pad1)
- C5 pad 2: Net-(C1-Pad2) -> Net-(C20-Pad1)
- C7 pad 1: Net-(U6--) -> Net-(U8--)
- C7 pad 2: Net-(C10-Pad2) -> Net-(C12-Pad2)
- C8 pad 1: Net-(U6--) -> Net-(U10--)
- C8 pad 2: Net-(C10-Pad2) -> Net-(C14-Pad2)
- C9 pad 1: Net-(U6--) -> Net-(U12--)
- C9 pad 2: Net-(C10-Pad2) -> Net-(C16-Pad2)
- R10 pad 1: Net-(C10-Pad2) -> Net-(C16-Pad2)
- R10 pad 2: Net-(C1-Pad1) -> Net-(C4-Pad1)
- R11 pad 1: Net-(C1-Pad2) -> Net-(C15-Pad1)
- R11 pad 2: Net-(U6--) -> Net-(U8--)
- R12 pad 1: Net-(C10-Pad2) -> Net-(C11-Pad2)
- R12 pad 2: Net-(C1-Pad1) -> Net-(C5-Pad1)
- R13 pad 1: Net-(C1-Pad2) -> Net-(C17-Pad1)
- R13 pad 2: Net-(U6--) -> Net-(U10--)
- R14 pad 1: Net-(C1-Pad2) -> Net-(C19-Pad1)
- R14 pad 2: Net-(U6--) -> Net-(U12--)
- R15 pad 1: Net-(C1-Pad2) -> Net-(C20-Pad1)
- R15 pad 2: Net-(U6--) -> Net-(U14--)
- R17 pad 1: Net-(U7-+) -> Net-(U9-+)
- R17 pad 2: Net-(C10-Pad2) -> Net-(C12-Pad2)
- R18 pad 1: Net-(U7-+) -> Net-(U11-+)
- R18 pad 2: Net-(C10-Pad2) -> Net-(C14-Pad2)
- R19 pad 1: Net-(U7-+) -> Net-(U13-+)
- R19 pad 2: Net-(C10-Pad2) -> Net-(C16-Pad2)
- R2 pad 1: Net-(R1-Pad1) -> Net-(R2-Pad1)
- R2 pad 2: Net-(R1-Pad2) -> Net-(R2-Pad2)
- R20 pad 1: Net-(U7-+) -> Net-(U15-+)
- R20 pad 2: Net-(C10-Pad2) -> Net-(C11-Pad2)
- R23 pad 1: Net-(U7--) -> Net-(U9--)
- R23 pad 2: Net-(U6-+) -> Net-(U8-+)
- R24 pad 1: Net-(U6-+) -> Net-(U8-+)
- R25 pad 1: Net-(U7--) -> Net-(U11--)
- R25 pad 2: Net-(U6-+) -> Net-(U10-+)
- R26 pad 1: Net-(U6-+) -> Net-(U10-+)
- R3 pad 1: Net-(R1-Pad1) -> Net-(R3-Pad1)
- R3 pad 2: Net-(R1-Pad2) -> Net-(R3-Pad2)
- R30 pad 1: Net-(U7--) -> Net-(U9--)
- R30 pad 2: Net-(C23-Pad2) -> Net-(C25-Pad2)
- R37 pad 1: Net-(C23-Pad2) -> Net-(C25-Pad2)
- R37 pad 2: Net-(U16-+) -> Net-(U17-+)
- R4 pad 1: Net-(R1-Pad1) -> Net-(R4-Pad1)
- R4 pad 2: Net-(R1-Pad2) -> Net-(R4-Pad2)
- R43 pad 1: Net-(C23-Pad1) -> Net-(C25-Pad1)
- R43 pad 2: Net-(U16--) -> Net-(U17--)
- R44 pad 1: Net-(U16--) -> Net-(U17--)
- R5 pad 1: Net-(R1-Pad1) -> Net-(R5-Pad1)
- R5 pad 2: Net-(R1-Pad2) -> Net-(R5-Pad2)
- R52 pad 1: Net-(C23-Pad1) -> Net-(C25-Pad1)
- R52 pad 2: Net-(U21-+) -> Net-(U22-+)
- R57 pad 1: Net-(U26-RW) -> Net-(U27-RW)
- R57 pad 2: Net-(C36-Pad1) -> Net-(C37-Pad1)
- R62 pad 1: Electrode Output 1 -> Electrode Output 2
- R7 pad 1: Net-(C10-Pad2) -> Net-(C12-Pad2)
- R7 pad 2: Net-(C1-Pad1) -> Net-(C2-Pad1)
- R8 pad 1: Net-(C10-Pad2) -> Net-(C14-Pad2)
- R8 pad 2: Net-(C1-Pad1) -> Net-(C3-Pad1)
- U10 pad 1: unconnected-(U6-NULL-Pad1) -> unconnected-(U10-NULL-Pad1)
- U10 pad 2: Net-(U6--) -> Net-(U10--)
- U10 pad 3: Net-(U6-+) -> Net-(U10-+)
- U10 pad 5: unconnected-(U6-NULL-Pad5) -> unconnected-(U10-NULL-Pad5)
- U10 pad 6: Net-(U6--) -> Net-(U10--)
- U10 pad 8: unconnected-(U6-NC-Pad8) -> unconnected-(U10-NC-Pad8)
- U11 pad 1: unconnected-(U7-NULL-Pad1) -> unconnected-(U11-NULL-Pad1)
- U11 pad 2: Net-(U7--) -> Net-(U11--)
- U11 pad 3: Net-(U7-+) -> Net-(U11-+)
- U11 pad 5: unconnected-(U7-NULL-Pad5) -> unconnected-(U11-NULL-Pad5)
- U11 pad 6: Net-(U7--) -> Net-(U11--)
- U11 pad 8: unconnected-(U7-NC-Pad8) -> unconnected-(U11-NC-Pad8)
- U12 pad 1: unconnected-(U6-NULL-Pad1) -> unconnected-(U12-NULL-Pad1)
- U12 pad 2: Net-(U6--) -> Net-(U12--)
- U12 pad 3: Net-(U6-+) -> Net-(U12-+)
- U12 pad 5: unconnected-(U6-NULL-Pad5) -> unconnected-(U12-NULL-Pad5)
- U12 pad 6: Net-(U6--) -> Net-(U12--)
- U12 pad 8: unconnected-(U6-NC-Pad8) -> unconnected-(U12-NC-Pad8)
- U13 pad 1: unconnected-(U7-NULL-Pad1) -> unconnected-(U13-NULL-Pad1)
- U13 pad 2: Net-(U7--) -> Net-(U13--)
- U13 pad 3: Net-(U7-+) -> Net-(U13-+)
- U13 pad 5: unconnected-(U7-NULL-Pad5) -> unconnected-(U13-NULL-Pad5)
- U13 pad 6: Net-(U7--) -> Net-(U13--)
- U13 pad 8: unconnected-(U7-NC-Pad8) -> unconnected-(U13-NC-Pad8)
- U14 pad 1: unconnected-(U6-NULL-Pad1) -> unconnected-(U14-NULL-Pad1)
- U14 pad 2: Net-(U6--) -> Net-(U14--)
- U14 pad 3: Net-(U6-+) -> Net-(U14-+)
- U14 pad 5: unconnected-(U6-NULL-Pad5) -> unconnected-(U14-NULL-Pad5)
- U14 pad 6: Net-(U6--) -> Net-(U14--)
- U14 pad 8: unconnected-(U6-NC-Pad8) -> unconnected-(U14-NC-Pad8)
- U15 pad 1: unconnected-(U7-NULL-Pad1) -> unconnected-(U15-NULL-Pad1)
- U15 pad 2: Net-(U7--) -> Net-(U15--)
- U15 pad 3: Net-(U7-+) -> Net-(U15-+)
- U15 pad 5: unconnected-(U7-NULL-Pad5) -> unconnected-(U15-NULL-Pad5)
- U15 pad 6: Net-(U7--) -> Net-(U15--)
- U15 pad 8: unconnected-(U7-NC-Pad8) -> unconnected-(U15-NC-Pad8)
- U17 pad 1: unconnected-(U16-NULL-Pad1) -> unconnected-(U17-NULL-Pad1)
- U17 pad 2: Net-(U16--) -> Net-(U17--)
- U17 pad 3: Net-(U16-+) -> Net-(U17-+)
- U17 pad 5: unconnected-(U16-NULL-Pad5) -> unconnected-(U17-NULL-Pad5)
- U17 pad 6: Net-(C23-Pad1) -> Net-(C25-Pad1)
- U17 pad 8: unconnected-(U16-NC-Pad8) -> unconnected-(U17-NC-Pad8)
- U2 pad 1: Net-(R1-Pad1) -> Net-(R2-Pad1)
- U2 pad 3: Electrode1 -> Electrode2
- U2 pad 6: Net-(C1-Pad1) -> Net-(C2-Pad1)
- U2 pad 8: Net-(R1-Pad2) -> Net-(R2-Pad2)
- U22 pad 1: unconnected-(U21-NULL-Pad1) -> unconnected-(U22-NULL-Pad1)
- U22 pad 2: Net-(U21--) -> Net-(U22--)
- U22 pad 3: Net-(U21-+) -> Net-(U22-+)
- U22 pad 5: unconnected-(U21-NULL-Pad5) -> unconnected-(U22-NULL-Pad5)
- U22 pad 6: Net-(C36-Pad1) -> Net-(C37-Pad1)
- U22 pad 8: unconnected-(U21-NC-Pad8) -> unconnected-(U22-NC-Pad8)
- U27 pad 1: unconnected-(U26-~{RST}-Pad1) -> unconnected-(U27-~{RST}-Pad1)
- U27 pad 12: CS 1 -> CS 2
- U27 pad 13: unconnected-(U26-SDO-Pad13) -> unconnected-(U27-SDO-Pad13)
- U27 pad 14: unconnected-(U26-RDY-Pad14) -> unconnected-(U27-RDY-Pad14)
- U27 pad 3: Net-(U21--) -> Net-(U22--)
- U27 pad 4: Net-(U26-RW) -> Net-(U27-RW)
- U27 pad 7: unconnected-(U26-EXT_CAP-Pad7) -> unconnected-(U27-EXT_CAP-Pad7)
- U3 pad 1: Net-(R1-Pad1) -> Net-(R3-Pad1)
- U3 pad 3: Electrode1 -> Electrode3
- U3 pad 6: Net-(C1-Pad1) -> Net-(C3-Pad1)
- U3 pad 8: Net-(R1-Pad2) -> Net-(R3-Pad2)
- U31 pad 10: CS 4 -> unconnected-(U31-8_TX2_IN1-Pad10)
- U31 pad 11: CS 3 -> unconnected-(U31-9_OUT1C-Pad11)
- U31 pad 12: CS 2 -> unconnected-(U31-10_CS_MQSR-Pad12)
- U31 pad 4: CS 10 -> unconnected-(U31-2_OUT2-Pad4)
- U31 pad 5: CS 9 -> unconnected-(U31-3_LRCLK2-Pad5)
- U31 pad 6: CS 8 -> unconnected-(U31-4_BCLK2-Pad6)
- U31 pad 7: CS 7 -> unconnected-(U31-5_IN2-Pad7)
- U31 pad 8: CS 6 -> unconnected-(U31-6_OUT1D-Pad8)
- U31 pad 9: CS 5 -> unconnected-(U31-7_RX2_OUT1A-Pad9)
- U4 pad 1: Net-(R1-Pad1) -> Net-(R4-Pad1)
- U4 pad 3: Electrode1 -> Electrode4
- U4 pad 6: Net-(C1-Pad1) -> Net-(C4-Pad1)
- U4 pad 8: Net-(R1-Pad2) -> Net-(R4-Pad2)
- U5 pad 1: Net-(R1-Pad1) -> Net-(R5-Pad1)
- U5 pad 3: Electrode1 -> Electrode5
- U5 pad 6: Net-(C1-Pad1) -> Net-(C5-Pad1)
- U5 pad 8: Net-(R1-Pad2) -> Net-(R5-Pad2)
- U8 pad 1: unconnected-(U6-NULL-Pad1) -> unconnected-(U8-NULL-Pad1)
- U8 pad 2: Net-(U6--) -> Net-(U8--)
- U8 pad 3: Net-(U6-+) -> Net-(U8-+)
- U8 pad 5: unconnected-(U6-NULL-Pad5) -> unconnected-(U8-NULL-Pad5)
- U8 pad 6: Net-(U6--) -> Net-(U8--)
- U8 pad 8: unconnected-(U6-NC-Pad8) -> unconnected-(U8-NC-Pad8)
- U9 pad 1: unconnected-(U7-NULL-Pad1) -> unconnected-(U9-NULL-Pad1)
- U9 pad 2: Net-(U7--) -> Net-(U9--)
- U9 pad 3: Net-(U7-+) -> Net-(U9-+)
- U9 pad 5: unconnected-(U7-NULL-Pad5) -> unconnected-(U9-NULL-Pad5)
- U9 pad 6: Net-(U7--) -> Net-(U9--)
- U9 pad 8: unconnected-(U7-NC-Pad8) -> unconnected-(U9-NC-Pad8)
Routing:
- net Net-(U6--): track 20.7 -> 124.1 mm, vias 2 -> 12
- net Net-(C10-Pad2): track 10.1 -> 60.5 mm
- net Net-(U6-+): track 12.4 -> 49.6 mm
- net Net-(U8--): track 0.00 -> 21.4 mm, vias 0 -> 2
- net Net-(U14--): track 0.00 -> 21.1 mm, vias 0 -> 2
- net Net-(U12--): track 0.00 -> 21.1 mm, vias 0 -> 2
- net Net-(U10--): track 0.00 -> 19.9 mm
- net Net-(C27-Pad1): track 0.00 -> 17.3 mm
- net Net-(C29-Pad1): track 0.00 -> 17.3 mm
- net Net-(C25-Pad1): track 0.00 -> 17.3 mm
- net Net-(C30-Pad1): track 0.00 -> 17.3 mm
- net Net-(C54-Pad1): track 0.00 -> 17.3 mm
- net Net-(C58-Pad1): track 0.00 -> 17.3 mm
- net Net-(C52-Pad1): track 0.00 -> 17.3 mm
- net Net-(C56-Pad1): track 0.00 -> 17.3 mm
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Other:
- board size 109.2 x 64.8 mm -> 108 x 130.8 mm
