File: Kicad Files/Heating Circuit/Heating Circuit.kicad_pcb (KiCad board)
At the start: 2 copper layers, 73.5 x 78 mm, 8 parts, among them J1 XT60_F_16.6V, J2 XT60_F_Heater, J3 XT60_F_Thermocouple, Q1 BUK9M52-40EX, U1 MAX31855KASA+T

Commit message: Added silkscreen and mounting holes
Parts:
- added REF**: MountingHole_2.2mm_M2, MountingHole:MountingHole_2.2mm_M2, F.Cu at (154.0, 104.0)
- added REF**: MountingHole_2.2mm_M2, MountingHole:MountingHole_2.2mm_M2, F.Cu at (154.0, 176.0)
- added REF**: MountingHole_2.2mm_M2, MountingHole:MountingHole_2.2mm_M2, F.Cu at (87.0, 176.0)
- added REF**: MountingHole_2.2mm_M2, MountingHole:MountingHole_2.2mm_M2, F.Cu at (87.0, 104.0)
Other:
- board size 73.5 x 78 mm -> 73 x 78 mm
- board text added: "Heating Circuit v1.0"

Commit message: Added ground plane
Routing:
- net MISO_thermocouple: track 0.00 -> 36.4 mm
- added copper zone on B.Cu, net GND_16.4V
- added copper zone on F.Cu, net GND_16.4V
Changed lines of the file:
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@@
 		(tags "Arduino Nano")
 		(property "Reference" "A1"
-			(at 7.62 -5.08 360)
+			(at 7.62 -5.08 0)
 			(layer "F.SilkS")
 			(effects
@@
 		(tags "RC Connector XT60")
 		(property "Reference" "J3"
-			(at 3.6 -17.5 360)
+			(at 3.6 -17.5 0)
 			(layer "F.SilkS")
 			(effects
@@
 		)
 		(property "Value" "XT60_F_Thermocouple"
-			(at 3.6 4 360)
+			(at 3.6 4 0)
 			(layer "F.Fab")
 			(effects
@@
 		)
 		(fp_text user "-"
-			(at -2.8 2.5 360)
+			(at -2.8 2.5 0)
 			(layer "F.SilkS")
 			(effects
@@
 		)
 		(fp_text user "+"
-			(at 9.5 2.5 360)
+			(at 9.5 2.5 0)
 			(layer "F.SilkS")
 			(effects
@@
 		)
 		(fp_text user "${REFERENCE}"
-			(at 3.6 -3.6 360)
+			(at 3.6 -3.6 0)
 			(layer "F.Fab")
 			(effects
@@
 		(tags "RC Connector XT60")
 		(property "Reference" "J2"
-			(at 3.6 -17.5 360)
+			(at 3.6 -17.5 0)
 			(layer "F.SilkS")
 			(effects
@@
 		)
 		(property "Value" "XT60_F_Heater"
-			(at 3.6 3.85 360)
+			(at 3.6 3.85 0)
 			(layer "F.Fab")
 			(effects
@@
 		)
 		(fp_text user "+"
-			(at 9.5 2.5 360)
+			(at 9.5 2.5 0)
 			(layer "F.SilkS")
 			(effects
@@
 		)
 		(fp_text user "-"
-			(at -2.8 2.5 360)
+			(at -2.8 2.5 0)
 			(layer "F.SilkS")
 			(effects
@@
 		)
 		(fp_text user "${REFERENCE}"
-			(at 3.6 -3.6 360)
+			(at 3.6 -3.6 0)
 			(layer "F.Fab")
 			(effects
@@
 		(tags "resistor")
 		(property "Reference" "R1"
-			(at 0 -1.65 360)
+			(at 0 -1.65 0)
 			(layer "F.SilkS")
 			(effects
@@
 		)
 		(property "Value" "100"
-			(at 0 1.65 360)
+			(at 0 1.65 0)
 			(layer "F.Fab")
 			(effects
@@
 		)
 		(fp_text user "${REFERENCE}"
-			(at 0 0 360)
+			(at 0 0 0)
 			(layer "F.Fab")
 			(effects
@@
 		)
 		(property "Value" "XT60_F_16.6V"
-			(at -5.9 -7.65 360)
+			(at -5.9 -7.65 0)
 			(layer "F.Fab")
 			(effects
@@
 		(tags "resistor")
 		(property "Reference" "R2"
-			(at 0 -1.65 360)
+			(at 0 -1.65 0)
 			(layer "F.SilkS")
 			(effects
@@
 		)
 		(property "Value" "10k"
-			(at 0 1.65 360)
+			(at 0 1.65 0)
 			(layer "F.Fab")
 			(effects
@@
 		)
 		(fp_text user "${REFERENCE}"
-			(at 0 0 360)
+			(at 0 0 0)
 			(layer "F.Fab")
 			(effects
@@
 		(tags "LFPAK33 SOT-1210")
 		(property "Reference" "Q1"
-			(at 0 -2.55 360)
+			(at 0 -2.55 0)
 			(layer "F.SilkS")
 			(effects
@@
 	)
 	(segment
+		(start 149.5 103)
+		(end 149.5 112.14)
+		(width 0.2)
+		(layer "F.Cu")
+		(net 2)
+	)
+	(segment
+		(start 134.0527 102.5)
+		(end 149 102.5)
+		(width 0.2)
+		(layer "F.Cu")
+		(net 2)
+	)
+	(segment
+		(start 149 102.5)
+		(end 149.5 103)
+		(width 0.2)
+		(layer "F.Cu")
+		(net 2)
+	)
+	(segment
+		(start 126.1877 110.365)
+		(end 134.0527 102.5)
+		(width 0.2)
+		(layer "F.Cu")
+		(net 2)
+	)
+	(segment
+		(start 125.72415 110.365)
+		(end 126.1877 110.365)
+		(width 0.2)
+		(layer "F.Cu")
+		(net 2)
+	)
+	(segment
 		(start 126.1877 111.635)
 		(end 133.8227 104)
@@
 		(net 36)
 	)
+	(zone
+		(net 4)
+		(net_name "GND_16.4V")
+		(layers "F&B.Cu")
+		(hatch edge 0.5)
+		(connect_pads
+			(clearance 0.5)
+		)
+		(min_thickness 0.25)
+		(filled_areas_thickness no)
+		(fill yes
+			(thermal_gap 0.5)
+			(thermal_bridge_width 0.5)
+		)
+		(polygon
+			(pts
+				(xy 74.5 87.5) (xy 71.5 186) (xy 170 184.5) (xy 168.5 87.5) (xy 70 93) (xy 69.5 93.5)
+			)
+		)
+	)
 )

Commit message: Heater Checked
Connections:
- net Net-(J1-Pin_2) renamed VCC_heater
- J2 pad 1: Net-(J2-Pin_1) -> GND_16.4V
- Q1 pad 1: Net-(J2-Pin_1) -> GND_16.4V
- Q1 pad 2: Net-(J2-Pin_1) -> GND_16.4V
- Q1 pad 3: Net-(J2-Pin_1) -> GND_16.4V
Routing:
- net GND_16.4V: track 110.4 -> 129.1 mm, vias 0 -> 3
- net Net-(J2-Pin_1): track 14.4 -> 0.00 mm
Changed lines of the file:
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@@
 	(net 28 "unconnected-(A1-A3-Pad22)")
 	(net 29 "unconnected-(A1-AREF-Pad18)")
-	(net 30 "Net-(J1-Pin_2)")
+	(net 30 "VCC_heater")
 	(net 31 "Net-(J1-Pin_1)")
 	(net 32 "Net-(J3-Pin_1)")
@@
 	(net 34 "Net-(Q1-G)")
 	(net 35 "unconnected-(U1-DNC-Pad8)")
-	(net 36 "Net-(J2-Pin_1)")
 	(footprint "Module:Arduino_Nano"
 		(layer "F.Cu")
@@
 			(net 18 "unconnected-(A1-D1{slash}TX-Pad1)")
 			(pinfunction "D1/TX")
-			(pintype "bidirectional")
+			(pintype "bidirectional+no_connect")
 		)
 		(pad "2" thru_hole oval
@@
 			(net 27 "unconnected-(A1-D0{slash}RX-Pad2)")
 			(pinfunction "D0/RX")
-			(pintype "bidirectional")
+			(pintype "bidirectional+no_connect")
 		)
 		(pad "3" thru_hole oval
@@
 			(net 14 "unconnected-(A1-~{RESET}-Pad3)")
 			(pinfunction "~{RESET}")
-			(pintype "input")
+			(pintype "input+no_connect")
 		)
 		(pad "4" thru_hole oval
@@
 			(net 10 "unconnected-(A1-D2-Pad5)")
 			(pinfunction "D2")
-			(pintype "bidirectional")
+			(pintype "bidirectional+no_connect")
 		)
 		(pad "6" thru_hole oval
@@
 			(net 16 "unconnected-(A1-D3-Pad6)")
 			(pinfunction "D3")
-			(pintype "bidirectional")
+			(pintype "bidirectional+no_connect")
 		)
 		(pad "7" thru_hole oval
@@
 			(net 1 "unconnected-(A1-D4-Pad7)")
 			(pinfunction "D4")
-			(pintype "bidirectional")
+			(pintype "bidirectional+no_connect")
 		)
 		(pad "8" thru_hole oval
@@
 			(net 20 "unconnected-(A1-D5-Pad8)")
 			(pinfunction "D5")
-			(pintype "bidirectional")
+			(pintype "bidirectional+no_connect")
 		)
 		(pad "9" thru_hole oval
@@
 			(net 22 "unconnected-(A1-D6-Pad9)")
 			(pinfunction "D6")
-			(pintype "bidirectional")
+			(pintype "bidirectional+no_connect")
 		)
 		(pad "10" thru_hole oval
@@
 			(net 15 "unconnected-(A1-D7-Pad10)")
 			(pinfunction "D7")
-			(pintype "bidirectional")
+			(pintype "bidirectional+no_connect")
 		)
 		(pad "11" thru_hole oval
@@
 			(net 11 "unconnected-(A1-D8-Pad11)")
 			(pinfunction "D8")
-			(pintype "bidirectional")
+			(pintype "bidirectional+no_connect")
 		)
 		(pad "12" thru_hole oval
@@
 			(net 6 "unconnected-(A1-D9-Pad12)")
 			(pinfunction "D9")
-			(pintype "bidirectional")
+			(pintype "bidirectional+no_connect")
 		)
 		(pad "13" thru_hole oval
@@
 			(net 29 "unconnected-(A1-AREF-Pad18)")
 			(pinfunction "AREF")
-			(pintype "input")
+			(pintype "input+no_connect")
 		)
 		(pad "19" thru_hole oval
@@
 			(net 19 "unconnected-(A1-A0-Pad19)")
 			(pinfunction "A0")
-			(pintype "bidirectional")
+			(pintype "bidirectional+no_connect")
 		)
 		(pad "20" thru_hole oval
@@
 			(net 13 "unconnected-(A1-A1-Pad20)")
 			(pinfunction "A1")
-			(pintype "bidirectional")
+			(pintype "bidirectional+no_connect")
 		)
 		(pad "21" thru_hole oval
@@
 			(net 24 "unconnected-(A1-A2-Pad21)")
 			(pinfunction "A2")
-			(pintype "bidirectional")
+			(pintype "bidirectional+no_connect")
 		)
 		(pad "22" thru_hole oval
@@
 			(net 28 "unconnected-(A1-A3-Pad22)")
 			(pinfunction "A3")
-			(pintype "bidirectional")
+			(pintype "bidirectional+no_connect")
 		)
 		(pad "23" thru_hole oval
@@
 			(net 5 "unconnected-(A1-A4-Pad23)")
 			(pinfunction "A4")
-			(pintype "bidirectional")
+			(pintype "bidirectional+no_connect")
 		)
 		(pad "24" thru_hole oval
@@
 			(net 9 "unconnected-(A1-A5-Pad24)")
 			(pinfunction "A5")
-			(pintype "bidirectional")
+			(pintype "bidirectional+no_connect")
 		)
 		(pad "25" thru_hole oval
@@
 			(net 25 "unconnected-(A1-A6-Pad25)")
 			(pinfunction "A6")
-			(pintype "bidirectional")
+			(pintype "bidirectional+no_connect")
 		)
 		(pad "26" thru_hole oval
@@
 			(net 23 "unconnected-(A1-A7-Pad26)")
 			(pinfunction "A7")
-			(pintype "bidirectional")
+			(pintype "bidirectional+no_connect")
 		)
 		(pad "27" thru_hole oval
@@
 			(net 26 "unconnected-(A1-+5V-Pad27)")
 			(pinfunction "+5V")
-			(pintype "power_out")
+			(pintype "power_out+no_connect")
 		)
 		(pad "28" thru_hole oval
@@
 			(net 8 "unconnected-(A1-~{RESET}-Pad28)")
 			(pinfunction "~{RESET}")
-			(pintype "input")
+			(pintype "input+no_connect")
 		)
 		(pad "29" thru_hole oval
@@
 			(net 7 "unconnected-(A1-VIN-Pad30)")
 			(pinfunction "VIN")
-			(pintype "power_in")
+			(pintype "power_in+no_connect")
 		)
 		(model "${KICAD8_3DMODEL_DIR}/Module.3dshapes/Arduino_Nano_WithMountingHoles.wrl"
@@
 			(remove_unused_layers no)
 			(roundrect_rratio 0.25)
-			(net 36 "Net-(J2-Pin_1)")
+			(net 4 "GND_16.4V")
 			(pinfunction "Pin_1")
 			(pintype "passive")
@@
 			(layers "*.Cu" "*.Mask")
 			(remove_unused_layers no)
-			(net 30 "Net-(J1-Pin_2)")
+			(net 30 "VCC_heater")
 			(pinfunction "Pin_2")
 			(pintype "passive")
@@
 			(layers "*.Cu" "*.Mask")
 			(remove_unused_layers no)
-			(net 30 "Net-(J1-Pin_2)")
+			(net 30 "VCC_heater")
 			(pinfunction "Pin_2")
 			(pintype "passive")
@@
 			(layers "F.Cu" "F.Mask")
 			(roundrect_rratio 0.25)
-			(net 36 "Net-(J2-Pin_1)")
+			(net 4 "GND_16.4V")
 			(pinfunction "S")
 			(pintype "passive")
@@
 			(layers "F.Cu" "F.Mask")
 			(roundrect_rratio 0.25)
-			(net 36 "Net-(J2-Pin_1)")
+			(net 4 "GND_16.4V")
 			(pinfunction "S")
 			(pintype "passive")
@@
 			(layers "F.Cu" "F.Mask")
 			(roundrect_rratio 0.25)
-			(net 36 "Net-(J2-Pin_1)")
+			(net 4 "GND_16.4V")
 			(pinfunction "S")
 			(pintype "passive")
@@
 	)
 	(segment
+		(start 118.18 160.651)
+		(end 118.18 161.301)
+		(width 0.2)
+		(layer "F.Cu")
+		(net 4)
+	)
+	(segment
+		(start 144.78 144.8)
+		(end 144.42 145.16)
+		(width 0.2)
+		(layer "F.Cu")
+		(net 4)
+	)
+	(segment
+		(start 108.401 160.651)
+		(end 105.1 157.35)
+		(width 0.2)
+		(layer "F.Cu")
+		(net 4)
+	)
+	(segment
 		(start 104.905 109.095)
 		(end 92 122)
@@
 	(segment
 		(start 149.5 140.08)
-		(end 144.42 145.16)
+		(end 144.8 144.78)
+		(width 0.2)
+		(layer "F.Cu")
+		(net 4)
+	)
+	(segment
+		(start 144.8 144.78)
+		(end 144.78 144.78)
+		(width 0.2)
+		(layer "F.Cu")
+		(net 4)
+	)
+	(segment
+		(start 118.18 160.651)
+		(end 108.401 160.651)
+		(width 0.2)
+		(layer "F.Cu")
+		(net 4)
+	)
+	(segment
+		(start 116.179 161.951)
+		(end 115.57 162.56)
+		(width 0.2)
+		(layer "F.Cu")
+		(net 4)
+	)
+	(segment
+		(start 144.78 144.78)
+		(end 144.78 144.8)
 		(width 0.2)
 		(layer "F.Cu")
@@
 	)
 	(segment
+		(start 118.18 161.301)
+		(end 118.18 161.951)
+		(width 0.2)
+		(layer "F.Cu")
+		(net 4)
+	)
+	(segment
+		(start 118.18 161.951)
+		(end 116.179 161.951)
+		(width 0.2)
+		(layer "F.Cu")
+		(net 4)
+	)
+	(segment
 		(start 120.27585 109.095)
 		(end 104.905 109.095)
@@
 		(net 4)
 	)
+	(via
+		(at 144.78 144.78)
+		(size 0.6)
+		(drill 0.3)
+		(layers "F.Cu" "B.Cu")
+		(net 4)
+	)
+	(via
+		(at 100.33 153.67)
+		(size 0.6)
+		(drill 0.3)
+		(layers "F.Cu" "B.Cu")
+		(free yes)
+		(net 4)
+	)
+	(via
+		(at 115.57 162.56)
+		(size 0.6)
+		(drill 0.3)
+		(layers "F.Cu" "B.Cu")
+		(net 4)
+	)
 	(segment
 		(start 134.26 112.14)
@@
 		(net 34)
 	)
-	(segment
-		(start 108.401 160.651)
-		(end 105.1 157.35)
-		(width 0.2)
-		(layer "F.Cu")
-		(net 36)
-	)
-	(segment
-		(start 118.18 160.651)
-		(end 108.401 160.651)
-		(width 0.2)
-		(layer "F.Cu")
-		(net 36)
-	)
 	(zone

Commit message: Fixed PWM direction, rerouted PCB trades
Parts:
- removed the REF** at (154.0, 104.0)
- removed the REF** at (154.0, 176.0)
- removed the REF** at (87.0, 176.0)
- removed the REF** at (87.0, 104.0)
- added REF**: MountingHole_2.2mm_M2_DIN965_Pad, MountingHole:MountingHole_2.2mm_M2_DIN965_Pad, F.Cu at (170.0, 151.5)
- added REF**: MountingHole_2.2mm_M2_DIN965_Pad, MountingHole:MountingHole_2.2mm_M2_DIN965_Pad, F.Cu at (170.0, 109.5)
- added REF**: MountingHole_2.2mm_M2_DIN965_Pad, MountingHole:MountingHole_2.2mm_M2_DIN965_Pad, F.Cu at (93.5, 109.5)
- added REF**: MountingHole_2.2mm_M2_DIN965_Pad, MountingHole:MountingHole_2.2mm_M2_DIN965_Pad, F.Cu at (93.5, 151.5)
- moved A1 62.9 mm to (97.9, 111.7), turned to 0 degrees
- moved J3 57.6 mm to (155.5, 124.5)
- moved J2 46.5 mm to (137.9, 124.5), turned to 0 degrees
- moved J1 40.1 mm to (120.4, 124.5), turned to 0 degrees
- moved U1 34.2 mm to (119.5, 145.0), turned to -90 degrees
- moved Q1 30.2 mm to (124.9, 131.9), turned to -90 degrees
- moved R2 23.1 mm to (117.1, 130.0), turned to 180 degrees
- moved R1 12.7 mm to (117.1, 135.5)
Connections:
- net VCC_heater renamed +16.4V
- J1 pad 1: Net-(J1-Pin_1) -> GND_16.4V
- Q1 pad 5: Net-(J1-Pin_1) -> GND_16.4V
- R1 pad 1: Net-(Q1-G) -> PWM_heater
- R1 pad 2: PWM_heater -> Net-(Q1-G)
- R2 pad 2: Net-(J1-Pin_1) -> GND_16.4V
Routing:
- net GND_16.4V: track 129.1 -> 62.8 mm, vias 3 -> 0
- net Net-(Q1-G): track 61.4 -> 11.5 mm
- net PWM_heater: track 71.0 -> 21.4 mm
- net Net-(J3-Pin_2): track 20.0 -> 50.1 mm
- net Net-(J1-Pin_1): track 23.6 -> 0.00 mm
- net +16.4V: track 41.8 -> 19.5 mm
- net CS_thermocouple: track 36.2 -> 22.5 mm
- net MISO_thermocouple: track 36.4 -> 23.5 mm
- net 3.3V_ard: track 14.7 -> 5.43 mm
- net Net-(J3-Pin_1): track 39.0 -> 44.3 mm
- net CLK: track 8.85 -> 4.63 mm
Other:
- board size 73 x 78 mm -> 84.5 x 49.5 mm
- board text removed: "Heating Circuit v1.0"
