File: Kicad Files/Heating Circuit/Heating Circuit.kicad_pcb (KiCad board)
At the start: 2 copper layers, 84.5 x 49.5 mm, 12 parts, among them J1 XT60_F_16.6V, J2 XT60_F_Heater, J3 XT60_F_Thermocouple, Q1 BUK9M52-40EX, U1 MAX31855KASA+T

Commit message: added thicker traces for heater power
Routing:
- net +16.4V: track 19.5 -> 20.2 mm
Changed lines of the file:
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@@
 	)
 	(setup
+		(stackup
+			(layer "F.SilkS"
+				(type "Top Silk Screen")
+			)
+			(layer "F.Paste"
+				(type "Top Solder Paste")
+			)
+			(layer "F.Mask"
+				(type "Top Solder Mask")
+				(thickness 0.01)
+			)
+			(layer "F.Cu"
+				(type "copper")
+				(thickness 0.035)
+			)
+			(layer "dielectric 1"
+				(type "core")
+				(thickness 1.51)
+				(material "FR4")
+				(epsilon_r 4.5)
+				(loss_tangent 0.02)
+			)
+			(layer "B.Cu"
+				(type "copper")
+				(thickness 0.035)
+			)
+			(layer "B.Mask"
+				(type "Bottom Solder Mask")
+				(thickness 0.01)
+			)
+			(layer "B.Paste"
+				(type "Bottom Solder Paste")
+			)
+			(layer "B.SilkS"
+				(type "Bottom Silk Screen")
+			)
+			(copper_finish "None")
+			(dielectric_constraints no)
+		)
 		(pad_to_mask_clearance 0)
 		(allow_soldermask_bridges_in_footprints no)
@@
 		(start 130.111 132.279)
 		(end 137.925 124.465)
-		(width 0.2)
+		(width 1)
 		(layer "F.Cu")
 		(net 4)
@@
 		(start 124.549 130.339)
 		(end 124.549 128.639)
-		(width 0.2)
+		(width 0.5)
 		(layer "F.Cu")
 		(net 4)
@@
 		(start 120.375 119.565)
 		(end 120.375 124.465)
-		(width 0.2)
+		(width 1)
 		(layer "F.Cu")
 		(net 4)
@@
 		(start 113.165 114.215)
 		(end 103.005 114.215)
-		(width 0.2)
+		(width 1)
 		(layer "F.Cu")
 		(net 4)
@@
 		(start 113.165 114.215)
 		(end 115.025 114.215)
-		(width 0.2)
+		(width 1)
 		(layer "F.Cu")
 		(net 4)
@@
 		(start 124.874 132.279)
 		(end 130.111 132.279)
-		(width 0.2)
+		(width 1)
 		(layer "F.Cu")
 		(net 4)
@@
 		(start 115.025 114.215)
 		(end 120.375 119.565)
-		(width 0.2)
+		(width 1)
 		(layer "F.Cu")
 		(net 4)
@@
 		(start 116.175 128.665)
 		(end 116.175 130)
-		(width 0.2)
+		(width 1)
 		(layer "F.Cu")
 		(net 4)
@@
 		(start 120.375 124.465)
 		(end 116.175 128.665)
-		(width 0.2)
+		(width 0.5)
 		(layer "F.Cu")
 		(net 4)
@@
 		(start 124.549 128.639)
 		(end 120.375 124.465)
-		(width 0.2)
+		(width 0.5)
 		(layer "F.Cu")
 		(net 4)
@@
 		(start 103.005 114.215)
 		(end 97.925 119.295)
-		(width 0.2)
+		(width 1)
 		(layer "F.Cu")
 		(net 4)
@@
 		(start 113.875 138.5)
 		(end 101.58 138.5)
-		(width 0.2)
+		(width 0.5)
 		(layer "F.Cu")
 		(net 21)
@@
 		(start 101.58 138.5)
 		(end 97.925 142.155)
-		(width 0.2)
+		(width 0.5)
 		(layer "F.Cu")
 		(net 21)
@@
 		(start 116.175 136.2)
 		(end 113.875 138.5)
-		(width 0.2)
+		(width 0.5)
 		(layer "F.Cu")
 		(net 21)
@@
 	(segment
 		(start 127.575 124.465)
-		(end 129.925 122.115)
-		(width 0.2)
+		(end 130.825 121.215)
+		(width 1)
 		(layer "F.Cu")
 		(net 30)
 	)
 	(segment
-		(start 129.925 122.115)
-		(end 142.775 122.115)
-		(width 0.2)
+		(start 141.875 121.215)
+		(end 145.125 124.465)
+		(width 1)
 		(layer "F.Cu")
 		(net 30)
 	)
 	(segment
-		(start 142.775 122.115)
-		(end 145.125 124.465)
-		(width 0.2)
+		(start 130.825 121.215)
+		(end 141.875 121.215)
+		(width 1)
 		(layer "F.Cu")
 		(net 30)
@@
 		(start 118 135.5)
 		(end 118 130)
-		(width 0.2)
+		(width 0.5)
 		(layer "F.Cu")
 		(net 33)
@@
 		(start 118 130)
 		(end 120.997 130)
-		(width 0.2)
+		(width 0.5)
 		(layer "F.Cu")
 		(net 33)
@@
 		(start 120.997 130)
 		(end 121.336 130.339)
-		(width 0.2)
+		(width 0.5)
 		(layer "F.Cu")
 		(net 33)
@@
 		(start 123.899 130.339)
 		(end 121.336 130.339)
-		(width 0.2)
+		(width 0.5)
 		(layer "F.Cu")
 		(net 33)

Commit message: Merge branch 'main' of https://github.com/jadoo-tech/Exoskeleton_public
Connections:
- J1 pad : (no net) -> GND_16.4V
Routing:
- net GND_16.4V: track 62.8 -> 47.1 mm
Changed lines of the file:
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@@
 			(layers "*.Cu" "*.Mask")
 			(remove_unused_layers no)
+			(net 4 "GND_16.4V")
 		)
 		(pad "" thru_hole rect
@@
 	)
 	(segment
-		(start 130.111 132.279)
-		(end 137.925 124.465)
+		(start 116.175 128.665)
+		(end 116.175 130)
 		(width 1)
 		(layer "F.Cu")
@@
 	)
 	(segment
-		(start 124.549 130.339)
-		(end 124.549 128.639)
-		(width 0.5)
-		(layer "F.Cu")
-		(net 4)
-	)
-	(segment
 		(start 120.375 119.565)
 		(end 120.375 124.465)
@@
 	)
 	(segment
-		(start 113.165 114.215)
-		(end 103.005 114.215)
+		(start 120.375 124.865)
+		(end 125.849 130.339)
 		(width 1)
 		(layer "F.Cu")
@@
 	(segment
 		(start 113.165 114.215)
-		(end 115.025 114.215)
+		(end 103.005 114.215)
 		(width 1)
 		(layer "F.Cu")
@@
 	)
 	(segment
-		(start 124.874 132.279)
-		(end 130.111 132.279)
+		(start 113.165 114.215)
+		(end 115.025 114.215)
 		(width 1)
 		(layer "F.Cu")
@@
 	)
 	(segment
-		(start 116.175 128.665)
-		(end 116.175 130)
-		(width 1)
-		(layer "F.Cu")
-		(net 4)
-	)
-	(segment
 		(start 120.375 124.465)
 		(end 116.175 128.665)
-		(width 0.5)
+		(width 1)
 		(layer "F.Cu")
 		(net 4)
 	)
 	(segment
-		(start 124.549 128.639)
-		(end 120.375 124.465)
-		(width 0.5)
+		(start 120.375 124.465)
+		(end 120.375 124.865)
+		(width 1)
 		(layer "F.Cu")
 		(net 4)
@@
 		(start 113.875 138.5)
 		(end 101.58 138.5)
-		(width 0.5)
+		(width 0.2)
 		(layer "F.Cu")
 		(net 21)
@@
 		(start 101.58 138.5)
 		(end 97.925 142.155)
-		(width 0.5)
+		(width 0.2)
 		(layer "F.Cu")
 		(net 21)
@@
 		(start 116.175 136.2)
 		(end 113.875 138.5)
-		(width 0.5)
+		(width 0.2)
 		(layer "F.Cu")
 		(net 21)
@@
 	(segment
 		(start 118 130)
-		(end 120.997 130)
-		(width 0.5)
-		(layer "F.Cu")
-		(net 33)
-	)
-	(segment
-		(start 120.997 130)
-		(end 121.336 130.339)
+		(end 123.56 130)
 		(width 0.5)
 		(layer "F.Cu")
@@
 	)
 	(segment
-		(start 123.899 130.339)
-		(end 121.336 130.339)
+		(start 123.56 130)
+		(end 123.899 130.339)
 		(width 0.5)
 		(layer "F.Cu")
