File: Kicad Files/Heating Circuit/Heating Circuit.kicad_sch (KiCad schematic)
At the start: 8 parts, among them J1 XT60_F_16.6V, J2 XT60_F_Heater, J3 XT60_F_Thermocouple, Q1 BUK9M52-40EX, U1 MAX31855KASA+T

Commit message: Minor schematic changes
Connections:
- net GND_ard_3.3V is gone; now on net GND: U1.1 (GND)
Changed lines of the file:
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@@
 		)
 	)
-	(global_label "GND_ard_3.3V"
+	(global_label "GND_ard"
 		(shape input)
 		(at 162.56 105.41 180)
@@
 		)
 		(property "Intersheetrefs" "${INTERSHEET_REFS}"
-			(at 146.5725 105.41 0)
+			(at 151.6525 105.41 0)
 			(effects
 				(font

Commit message: Heater Checked
Connections:
- net GND: now also J2.1 (Pin_1), Q1.1 (S), Q1.2 (S), Q1.3 (S)
- net VCC_heater: now also J1.2 (Pin_2), J2.2 (Pin_2)
- net 3.3V_ard renamed +3.3V
- no-connect marks 0 -> 23
Changed lines of the file:
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@@
+	)
+	(junction
+		(at 85.09 146.05)
+		(diameter 0)
+		(color 0 0 0 0)
 	)
 	(junction
@@
 	)
 	(junction
+		(at 185.42 50.8)
+		(diameter 0)
+		(color 0 0 0 0)
+	)
+	(junction
 		(at 99.06 148.59)
+		(diameter 0)
+		(color 0 0 0 0)
+	)
+	(junction
+		(at 185.42 48.26)
 		(diameter 0)
 		(color 0 0 0 0)
@@
 		(color 0 0 0 0)
 	)
+	(no_connect
+		(at 111.76 125.73)
+	)
+	(no_connect
+		(at 96.52 90.17)
+	)
+	(no_connect
+		(at 86.36 120.65)
+	)
+	(no_connect
+		(at 111.76 100.33)
+	)
+	(no_connect
+		(at 111.76 130.81)
+	)
+	(no_connect
+		(at 86.36 118.11)
+	)
+	(no_connect
+		(at 86.36 107.95)
+	)
+	(no_connect
+		(at 111.76 118.11)
+	)
+	(no_connect
+		(at 86.36 105.41)
+	)
+	(no_connect
+		(at 86.36 115.57)
+	)
+	(no_connect
+		(at 111.76 133.35)
+	)
+	(no_connect
+		(at 86.36 123.19)
+	)
+	(no_connect
+		(at 111.76 120.65)
+	)
+	(no_connect
+		(at 111.76 102.87)
+	)
+	(no_connect
+		(at 111.76 115.57)
+	)
+	(no_connect
+		(at 86.36 102.87)
+	)
+	(no_connect
+		(at 86.36 110.49)
+	)
+	(no_connect
+		(at 86.36 113.03)
+	)
+	(no_connect
+		(at 86.36 100.33)
+	)
+	(no_connect
+		(at 111.76 110.49)
+	)
+	(no_connect
+		(at 111.76 123.19)
+	)
+	(no_connect
+		(at 111.76 128.27)
+	)
+	(no_connect
+		(at 104.14 90.17)
+	)
 	(wire
 		(pts
@@
 	(wire
 		(pts
-			(xy 189.23 50.8) (xy 179.07 50.8)
+			(xy 189.23 50.8) (xy 185.42 50.8)
 		)
 		(stroke
@@
 	(wire
 		(pts
+			(xy 185.42 44.45) (xy 185.42 48.26)
+		)
+		(stroke
+			(width 0)
+			(type default)
+		)
+	)
+	(wire
+		(pts
 			(xy 149.86 64.77) (xy 149.86 80.01)
 		)
@@
 	(wire
 		(pts
+			(xy 185.42 50.8) (xy 179.07 50.8)
+		)
+		(stroke
+			(width 0)
+			(type default)
+		)
+	)
+	(wire
+		(pts
 			(xy 139.7 62.23) (xy 144.78 62.23)
 		)
@@
 	(wire
 		(pts
-			(xy 101.6 77.47) (xy 101.6 90.17)
+			(xy 101.6 74.93) (xy 101.6 90.17)
 		)
 		(stroke
@@
 	(wire
 		(pts
+			(xy 82.55 146.05) (xy 85.09 146.05)
+		)
+		(stroke
+			(width 0)
+			(type default)
+		)
+	)
+	(wire
+		(pts
 			(xy 85.09 146.05) (xy 85.09 148.59)
 		)
@@
 	(wire
 		(pts
-			(xy 149.86 48.26) (xy 189.23 48.26)
+			(xy 149.86 48.26) (xy 185.42 48.26)
 		)
 		(stroke
@@
 	(wire
 		(pts
-			(xy 85.09 148.59) (xy 85.09 151.13)
+			(xy 85.09 148.59) (xy 85.09 152.4)
 		)
 		(stroke
@@
 	(wire
 		(pts
+			(xy 185.42 50.8) (xy 185.42 59.69)
+		)
+		(stroke
+			(width 0)
+			(type default)
+		)
+	)
+	(wire
+		(pts
+			(xy 185.42 48.26) (xy 189.23 48.26)
+		)
+		(stroke
+			(width 0)
+			(type default)
+		)
+	)
+	(wire
+		(pts
 			(xy 80.01 125.73) (xy 86.36 125.73)
 		)
@@
 	(global_label "VCC_heater"
 		(shape input)
-		(at 194.31 48.26 0)
+		(at 185.42 44.45 0)
 		(fields_autoplaced yes)
 		(effects
@@
 		)
 		(property "Intersheetrefs" "${INTERSHEET_REFS}"
-			(at 207.8785 48.26 0)
+			(at 198.9885 44.45 0)
 			(effects
 				(font
@@
 	(global_label "GND_heater"
 		(shape input)
-		(at 194.31 50.8 0)
+		(at 185.42 59.69 0)
 		(fields_autoplaced yes)
 		(effects
@@
 		)
 		(property "Intersheetrefs" "${INTERSHEET_REFS}"
-			(at 208.1204 50.8 0)
+			(at 199.2304 59.69 0)
 			(effects
 				(font
@@
 		(property "Intersheetrefs" "${INTERSHEET_REFS}"
 			(at 142.24 84.5675 90)
+			(effects
+				(font
+					(size 1.27 1.27)
+				)
+				(justify right)
+				(hide yes)
+			)
+		)
+	)
+	(global_label "GND_heater"
+		(shape input)
+		(at 82.55 146.05 180)
+		(fields_autoplaced yes)
+		(effects
+			(font
+				(size 1.27 1.27)
+			)
+			(justify right)
+		)
+		(property "Intersheetrefs" "${INTERSHEET_REFS}"
+			(at 68.7396 146.05 0)
 			(effects
 				(font
@@
 	(symbol
 		(lib_id "power:GND")
-		(at 85.09 151.13 0)
+		(at 85.09 152.4 0)
 		(unit 1)
 		(exclude_from_sim no)
@@
 		(fields_autoplaced yes)
 		(property "Reference" "#PWR01"
+			(at 85.09 158.75 0)
+			(effects
+				(font
+					(size 1.27 1.27)
+				)
+				(hide yes)
+			)
+		)
+		(property "Value" "GND"
 			(at 85.09 157.48 0)
 			(effects
@@
 					(size 1.27 1.27)
 				)
-				(hide yes)
-			)
-		)
-		(property "Value" "GND"
-			(at 85.09 156.21 0)
-			(effects
-				(font
-					(size 1.27 1.27)
-				)
 			)
 		)
 		(property "Footprint" ""
-			(at 85.09 151.13 0)
+			(at 85.09 152.4 0)
 			(effects
 				(font
@@
 		)
 		(property "Datasheet" ""
-			(at 85.09 151.13 0)
+			(at 85.09 152.4 0)
 			(effects
 				(font
@@
 		)
 		(property "Description" "Power symbol creates a global label with name \"GND\" , ground"
-			(at 85.09 151.13 0)
+			(at 85.09 152.4 0)
 			(effects
 				(font
@@
 					(unit 1)
 				)
+			)
+		)
+	)
+	(symbol
+		(lib_id "power:+3.3V")
+		(at 101.6 74.93 0)
+		(unit 1)
+		(exclude_from_sim no)
+		(in_bom yes)
+		(on_board yes)
+		(dnp no)
+		(fields_autoplaced yes)
+		(property "Reference" "#PWR02"
+			(at 101.6 78.74 0)
+			(effects
+				(font
+					(size 1.27 1.27)
+				)
+				(hide yes)
+			)
+		)
+		(property "Value" "+3.3V"
+			(at 101.6 69.85 0)
+			(effects
+				(font
+					(size 1.27 1.27)
+				)
+			)
+		)
+		(property "Footprint" ""
+			(at 101.6 74.93 0)
+			(effects
+				(font
+					(size 1.27 1.27)
+				)
+				(hide yes)
+			)
+		)
+		(property "Datasheet" ""
+			(at 101.6 74.93 0)
+			(effects
+				(font
+					(size 1.27 1.27)
+				)
+				(hide yes)
+			)
+		)
+		(property "Description" "Power symbol creates a global label with name \"+3.3V\""
+			(at 101.6 74.93 0)
+			(effects
+				(font
+					(size 1.27 1.27)
+				)
+				(hide yes)
+			)
+		)
+		(pin "1"
+		)
+		(instances
+			(project ""
+				(path "/897be0cd-1f22-4e2d-9992-bf172b338bf2"
+					(reference "#PWR02")
+					(unit 1)
+				)

Commit message: Fixed schematics
Connections:
- net VCC_heater is gone; now on net +16.4V: J1.2 (Pin_2), J2.2 (Pin_2)
- net GND: now also J1.1 (Pin_1), Q1.5 (D), R2.2
Changed lines of the file:
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@@
+	)
+	(junction
+		(at 149.86 68.58)
+		(diameter 0)
+		(color 0 0 0 0)
 	)
 	(junction
@@
 	)
 	(junction
+		(at 149.86 54.61)
+		(diameter 0)
+		(color 0 0 0 0)
+	)
+	(junction
 		(at 185.42 50.8)
 		(diameter 0)
@@
 	)
 	(junction
-		(at 142.24 64.77)
+		(at 144.78 68.58)
 		(diameter 0)
 		(color 0 0 0 0)
@@
 	(wire
 		(pts
-			(xy 142.24 64.77) (xy 142.24 73.66)
+			(xy 144.78 68.58) (xy 144.78 77.47)
 		)
 		(stroke
@@
 	(wire
 		(pts
-			(xy 149.86 64.77) (xy 149.86 80.01)
+			(xy 149.86 64.77) (xy 149.86 68.58)
+		)
+		(stroke
+			(width 0)
+			(type default)
+		)
+	)
+	(wire
+		(pts
+			(xy 149.86 54.61) (xy 149.86 62.23)
 		)
 		(stroke
@@
 	(wire
 		(pts
-			(xy 139.7 62.23) (xy 144.78 62.23)
+			(xy 138.43 54.61) (xy 149.86 54.61)
 		)
 		(stroke
@@
 	(wire
 		(pts
-			(xy 142.24 64.77) (xy 144.78 64.77)
+			(xy 144.78 68.58) (xy 149.86 68.58)
 		)
 		(stroke
@@
 	(wire
 		(pts
-			(xy 149.86 48.26) (xy 149.86 62.23)
+			(xy 149.86 48.26) (xy 149.86 54.61)
 		)
 		(stroke
@@
 	(wire
 		(pts
+			(xy 149.86 68.58) (xy 149.86 80.01)
+		)
+		(stroke
+			(width 0)
+			(type default)
+		)
+	)
+	(wire
+		(pts
 			(xy 186.69 74.93) (xy 191.77 74.93)
 		)
@@
 	(wire
 		(pts
-			(xy 139.7 64.77) (xy 142.24 64.77)
+			(xy 142.24 68.58) (xy 144.78 68.58)
 		)
 		(stroke
@@
 	(global_label "GND_16.4V"
 		(shape input)
-		(at 139.7 64.77 180)
+		(at 142.24 68.58 180)
 		(fields_autoplaced yes)
 		(effects
@@
 		)
 		(property "Intersheetrefs" "${INTERSHEET_REFS}"
-			(at 126.5548 64.77 0)
+			(at 129.0948 68.58 0)
 			(effects
 				(font
@@
 	(global_label "+16.4V"
 		(shape input)
-		(at 139.7 62.23 180)
+		(at 138.43 54.61 180)
 		(fields_autoplaced yes)
 		(effects
@@
 		)
 		(property "Intersheetrefs" "${INTERSHEET_REFS}"
-			(at 129.8205 62.23 0)
+			(at 128.5505 54.61 0)
 			(effects
 				(font
@@
 	(global_label "GND_ard"
 		(shape input)
-		(at 142.24 73.66 270)
+		(at 144.78 77.47 270)
 		(fields_autoplaced yes)
 		(effects
@@
 		)
 		(property "Intersheetrefs" "${INTERSHEET_REFS}"
-			(at 142.24 84.5675 90)
-			(effects
-				(font
+			(at 144.78 88.3775 90)
+			(effects
+				(font

Commit message: Fixed PWM direction, rerouted PCB trades
Connections:
- net PWM_heater: now also R1.1; no longer R1.2
- net at Q1.4 (G), R2.1: now also R1.2; no longer R1.1
Other:
- moved on the sheet: Q1, R1, R2
Changed lines of the file:
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@@
 	(paper "A4")
-	(junction
-		(at 179.07 80.01)
-		(diameter 0)
-		(color 0 0 0 0)
-	)
 	(junction
 		(at 85.09 146.05)
@@
 	)
 	(junction
+		(at 163.83 80.01)
+		(diameter 0)
+		(color 0 0 0 0)
+	)
+	(junction
 		(at 149.86 54.61)
 		(diameter 0)
@@
 	)
 	(junction
+		(at 170.18 74.93)
+		(diameter 0)
+		(color 0 0 0 0)
+	)
+	(junction
 		(at 85.09 148.59)
 		(diameter 0)
@@
 		(color 0 0 0 0)
 	)
-	(junction
-		(at 186.69 74.93)
-		(diameter 0)
-		(color 0 0 0 0)
-	)
 	(no_connect
 		(at 111.76 125.73)
@@
 	(wire
 		(pts
+			(xy 163.83 74.93) (xy 163.83 80.01)
+		)
+		(stroke
+			(width 0)
+			(type default)
+		)
+	)
+	(wire
+		(pts
 			(xy 179.07 50.8) (xy 179.07 69.85)
 		)
@@
 	(wire
 		(pts
-			(xy 179.07 80.01) (xy 181.61 80.01)
-		)
-		(stroke
-			(width 0)
-			(type default)
-		)
-	)
-	(wire
-		(pts
 			(xy 85.09 148.59) (xy 99.06 148.59)
 		)
@@
 	(wire
 		(pts
-			(xy 199.39 74.93) (xy 204.47 74.93)
-		)
-		(stroke
-			(width 0)
-			(type default)
-		)
-	)
-	(wire
-		(pts
 			(xy 149.86 68.58) (xy 149.86 80.01)
 		)
@@
 	(wire
 		(pts
-			(xy 186.69 74.93) (xy 191.77 74.93)
-		)
-		(stroke
-			(width 0)
-			(type default)
-		)
-	)
-	(wire
-		(pts
 			(xy 80.01 128.27) (xy 86.36 128.27)
 		)
@@
 	(wire
 		(pts
-			(xy 149.86 80.01) (xy 179.07 80.01)
+			(xy 149.86 80.01) (xy 163.83 80.01)
 		)
 		(stroke
@@
 	(wire
 		(pts
+			(xy 170.18 74.93) (xy 171.45 74.93)
+		)
+		(stroke
+			(width 0)
+			(type default)
+		)
+	)
+	(wire
+		(pts
+			(xy 168.91 74.93) (xy 170.18 74.93)
+		)
+		(stroke
+			(width 0)
+			(type default)
+		)
+	)
+	(wire
+		(pts
 			(xy 185.42 48.26) (xy 189.23 48.26)
 		)
@@
 	(wire
 		(pts
+			(xy 163.83 80.01) (xy 179.07 80.01)
+		)
+		(stroke
+			(width 0)
+			(type default)
+		)
+	)
+	(wire
+		(pts
+			(xy 170.18 71.12) (xy 170.18 74.93)
+		)
+		(stroke
+			(width 0)
+			(type default)
+		)
+	)
+	(wire
+		(pts
 			(xy 80.01 125.73) (xy 86.36 125.73)
 		)
@@
 	(wire
 		(pts
-			(xy 186.69 74.93) (xy 186.69 80.01)
+			(xy 166.37 63.5) (xy 170.18 63.5)
 		)
 		(stroke
@@
 	(global_label "PWM_heater"
 		(shape input)
-		(at 204.47 74.93 0)
-		(fields_autoplaced yes)
-		(effects
-			(font
-				(size 1.27 1.27)
-			)
-			(justify left)
-		)
-		(property "Intersheetrefs" "${INTERSHEET_REFS}"
-			(at 218.5827 74.93 0)
-			(effects
-				(font
-					(size 1.27 1.27)
-				)
-				(justify left)
+		(at 166.37 63.5 180)
+		(fields_autoplaced yes)
+		(effects
+			(font
+				(size 1.27 1.27)
+			)
+			(justify right)
+		)
+		(property "Intersheetrefs" "${INTERSHEET_REFS}"
+			(at 152.2573 63.5 0)
+			(effects
+				(font
+					(size 1.27 1.27)
+				)
+				(justify right)
 				(hide yes)
 			)
@@
 	(symbol
 		(lib_id "Transistor_FET:BUK9M52-40EX")
-		(at 181.61 74.93 180)
+		(at 176.53 74.93 0)
 		(unit 1)
 		(exclude_from_sim no)
@@
 		(on_board yes)
 		(dnp no)
-		(fields_autoplaced yes)
 		(property "Reference" "Q1"
-			(at 175.26 73.6599 0)
+			(at 182.88 73.6599 0)
 			(effects
 				(font
@@
 		)
 		(property "Value" "BUK9M52-40EX"
-			(at 175.26 76.1999 0)
+			(at 182.88 76.1999 0)
 			(effects
 				(font
@@
 		)
 		(property "Footprint" "Package_TO_SOT_SMD:LFPAK33"
-			(at 176.53 73.025 0)
+			(at 181.61 76.835 0)
 			(effects
 				(font
@@
 		)
 		(property "Datasheet" "https://assets.nexperia.com/documents/data-sheet/BUK9M52-40E.pdf"
-			(at 176.53 71.12 0)
+			(at 181.61 78.74 0)
 			(effects
 				(font
@@
 		)
 		(property "Description" "17.6A Id, 40V Vds, N-Channel TrenchMOS MOSFET, 40mOhm Ron, 4.5nC Qqd, -55 to 175 °C, LFPAK33"
-			(at 181.61 74.93 0)
+			(at 176.53 74.93 0)
 			(effects
 				(font
@@
 	(symbol
 		(lib_id "Device:R")
-		(at 195.58 74.93 90)
+		(at 170.18 67.31 0)
 		(unit 1)
 		(exclude_from_sim no)
@@
 		(dnp no)
 		(property "Reference" "R1"
-			(at 195.58 69.85 90)
+			(at 175.26 67.31 90)
 			(effects
 				(font
@@
 		)
 		(property "Value" "100"
-			(at 195.58 72.39 90)
+			(at 172.72 67.31 90)
 			(effects
 				(font
@@
 		)
 		(property "Footprint" "Resistor_SMD:R_0805_2012Metric"
-			(at 195.58 76.708 90)
+			(at 168.402 67.31 90)
 			(effects
 				(font
@@
 		)
 		(property "Datasheet" "~"
-			(at 195.58 74.93 0)
+			(at 170.18 67.31 0)
 			(effects
 				(font
@@
 		)
 		(property "Description" "Resistor"
-			(at 195.58 74.93 0)
+			(at 170.18 67.31 0)
 			(effects
 				(font
@@
 	(symbol
 		(lib_id "Device:R_Small")
-		(at 184.15 80.01 270)
+		(at 166.37 74.93 270)
 		(unit 1)
 		(exclude_from_sim no)
@@
 		(dnp no)
 		(property "Reference" "R2"
-			(at 184.15 82.296 90)
+			(at 166.37 77.216 90)
 			(effects
 				(font
@@
 		)
 		(property "Value" "10k"
-			(at 184.15 84.836 90)
+			(at 166.37 79.756 90)
 			(effects
 				(font
@@
 		)
 		(property "Footprint" "Resistor_SMD:R_0805_2012Metric"
-			(at 184.15 80.01 0)
+			(at 166.37 74.93 0)
 			(effects
 				(font
@@
 		)
 		(property "Datasheet" "~"
-			(at 184.15 80.01 0)
+			(at 166.37 74.93 0)
 			(effects
 				(font
@@
 		)
 		(property "Description" "Resistor, small symbol"
-			(at 184.15 80.01 0)
-			(effects
-				(font
+			(at 166.37 74.93 0)
+			(effects
+				(font
