File: Kicad Files/Heating Circuit/Limb_Circuit.kicad_pcb (KiCad board)
At the start: 2 copper layers, 84.5 x 49.5 mm, 12 parts, among them J1 XT60_F_16.6V, J2 XT60_F_Heater, J3 XT60_F_Thermocouple, Q1 BUK9M52-40EX, U1 MAX31855KASA+T

Commit message: adding gyroscope
Routing:
- net GND_16.4V: track 47.1 -> 65.2 mm
Changed lines of the file:
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@@
+	)
+	(segment
+		(start 137.925 127.575)
+		(end 133.221 132.279)
+		(width 1)
+		(layer "F.Cu")
+		(net 4)
+	)
+	(segment
+		(start 133.221 132.279)
+		(end 124.874 132.279)
+		(width 1)
+		(layer "F.Cu")
+		(net 4)
 	)
 	(segment
@@
 		(width 1)
 		(layer "F.Cu")
+		(net 4)
+	)
+	(segment
+		(start 137.925 124.465)
+		(end 137.925 127.575)
+		(width 1)
+		(layer "F.Cu")
