File: Kicad Files/Heating Circuit/Limb_Circuit.kicad_sch (KiCad schematic)
At the start: 8 parts, among them J1 XT60_F_16.6V, J2 XT60_F_Heater, J3 XT60_F_Thermocouple, Q1 BUK9M52-40EX, U1 MAX31855KASA+T

Commit message: adding gyroscope
Parts:
- added U2: LSM6DSL, Package_LGA:LGA-14_3x2.5mm_P0.5mm_LayoutBorder3x4y, symbol Sensor_Motion:LSM6DSL
Connections:
- net +3.3V: now also U2.5 (VDDIO), U2.8 (VDD)
- net GND: no longer J2.1 (Pin_1), Q1.5 (D)
- new net: U2.6 (GND), U2.7 (GND)
- new net GND_heater: J2.1 (Pin_1), Q1.5 (D)
Changed lines of the file:
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@@
 	(paper "A4")
-	(junction
-		(at 85.09 146.05)
-		(diameter 0)
-		(color 0 0 0 0)
-	)
 	(junction
 		(at 149.86 68.58)
@@
 		(color 0 0 0 0)
 	)
+	(junction
+		(at 153.67 132.08)
+		(diameter 0)
+		(color 0 0 0 0)
+	)
 	(no_connect
 		(at 111.76 125.73)
@@
 	(wire
 		(pts
+			(xy 153.67 125.73) (xy 153.67 132.08)
+		)
+		(stroke
+			(width 0)
+			(type default)
+		)
+	)
+	(wire
+		(pts
 			(xy 101.6 74.93) (xy 101.6 90.17)
 		)
@@
 	(wire
 		(pts
+			(xy 153.67 132.08) (xy 156.21 132.08)
+		)
+		(stroke
+			(width 0)
+			(type default)
+		)
+	)
+	(wire
+		(pts
 			(xy 163.83 74.93) (xy 163.83 80.01)
 		)
@@
 	(wire
 		(pts
+			(xy 156.21 132.08) (xy 156.21 135.89)
+		)
+		(stroke
+			(width 0)
+			(type default)
+		)
+	)
+	(wire
+		(pts
 			(xy 99.06 148.59) (xy 99.06 149.86)
 		)
@@
 	(wire
 		(pts
-			(xy 82.55 146.05) (xy 85.09 146.05)
-		)
-		(stroke
-			(width 0)
-			(type default)
-		)
-	)
-	(wire
-		(pts
 			(xy 85.09 146.05) (xy 85.09 148.59)
 		)
@@
 	(wire
 		(pts
+			(xy 153.67 132.08) (xy 153.67 135.89)
+		)
+		(stroke
+			(width 0)
+			(type default)
+		)
+	)
+	(wire
+		(pts
 			(xy 185.42 48.26) (xy 189.23 48.26)
 		)
@@
 		)
 	)
-	(global_label "GND_heater"
-		(shape input)
-		(at 82.55 146.05 180)
+	(global_label "3.3V_ard"
+		(shape input)
+		(at 153.67 125.73 180)
 		(fields_autoplaced yes)
 		(effects
@@
 		)
 		(property "Intersheetrefs" "${INTERSHEET_REFS}"
-			(at 68.7396 146.05 0)
+			(at 142.5206 125.73 0)
 			(effects
 				(font
@@
 					(unit 1)
 				)
+			)
+		)
+	)
+	(symbol
+		(lib_id "Sensor_Motion:LSM6DSL")
+		(at 153.67 151.13 0)
+		(unit 1)
+		(exclude_from_sim no)
+		(in_bom yes)
+		(on_board yes)
+		(dnp no)
+		(fields_autoplaced yes)
+		(property "Reference" "U2"
+			(at 155.8641 166.37 0)
+			(effects
+				(font
+					(size 1.27 1.27)
+				)
+				(justify left)
+			)
+		)
+		(property "Value" "LSM6DSL"
+			(at 155.8641 168.91 0)
+			(effects
+				(font
+					(size 1.27 1.27)
+				)
+				(justify left)
+			)
+		)
+		(property "Footprint" "Package_LGA:LGA-14_3x2.5mm_P0.5mm_LayoutBorder3x4y"
+			(at 143.51 168.91 0)
+			(effects
+				(font
+					(size 1.27 1.27)
+				)
+				(justify left)
+				(hide yes)
+			)
+		)
+		(property "Datasheet" "https://www.st.com/resource/en/datasheet/lsm6dsl.pdf"
+			(at 156.21 167.64 0)
+			(effects
+				(font
+					(size 1.27 1.27)
+				)
+				(hide yes)
+			)
+		)
+		(property "Description" "I2C/SPI, iNEMO inertial module: always-on 3D accelerometer and 3D gyroscope, 1.71V to 3.6V VCC"
+			(at 153.67 151.13 0)
+			(effects
+				(font
+					(size 1.27 1.27)
+				)
+				(hide yes)
+			)
+		)
+		(pin "8"
+		)
+		(pin "6"
+		)
+		(pin "4"
+		)
+		(pin "12"
+		)
+		(pin "2"
+		)
+		(pin "13"
+		)
+		(pin "5"
+		)
+		(pin "14"
+		)
+		(pin "1"
+		)
+		(pin "11"
+		)
+		(pin "9"
+		)
+		(pin "10"
+		)
+		(pin "3"
+		)
+		(pin "7"
+		)
+		(instances
+			(project ""
+				(path "/897be0cd-1f22-4e2d-9992-bf172b338bf2"
+					(reference "U2")
+					(unit 1)
+				)
