File: Kicad Files/Limb Circuit/Limb_Circuit.kicad_pcb (KiCad board)
At the start: 2 copper layers, 84.5 x 49.5 mm, 12 parts, among them J1 XT60_F_16.6V, J2 XT60_F_Heater, J3 XT60_F_Thermocouple, Q1 BUK9M52-40EX, U1 MAX31855KASA+T

Commit message: Added gyroscope
Parts:
- added C1: 0.1uF, Capacitor_SMD:C_0402_1005Metric, F.Cu at (134.0, 143.5)
- added C2: 0.1uF, Capacitor_SMD:C_0402_1005Metric, F.Cu at (133.5, 140.0)
- added R3: 10k, Resistor_SMD:R_0805_2012Metric, F.Cu at (129.1, 144.0)
- added U2: LSM6DSL, Package_LGA:LGA-14_3x2.5mm_P0.5mm_LayoutBorder3x4y, F.Cu at (129.2, 138.1)
- moved U1 7.78 mm to (125.8, 149.6), turned to 180 degrees
- moved R1 2.00 mm to (117.1, 133.5)
Connections:
- A1 pad 23: unconnected-(A1-A4-Pad23) -> SDA_gyro
- A1 pad 24: unconnected-(A1-A5-Pad24) -> SCL_gyro
- J1 pad : GND_16.4V -> (no net)
- J2 pad 1: GND_16.4V -> GND_heater
- Q1 pad 5: GND_16.4V -> GND_heater
Routing:
- net GND_16.4V: track 65.2 -> 121.5 mm
- net 3.3V_ard: track 5.43 -> 43.2 mm
- net SDA_gyro: track 0.00 -> 29.7 mm
- net SCL_gyro: track 0.00 -> 23.5 mm
- net GND_heater: track 0.00 -> 18.1 mm
- net PWM_heater: track 21.4 -> 38.2 mm
- net Net-(J3-Pin_1): track 44.3 -> 37.1 mm
- net CLK: track 4.63 -> 10.1 mm
- net Net-(J3-Pin_2): track 50.1 -> 44.8 mm
- net CS_thermocouple: track 22.5 -> 26.9 mm
- net Net-(U2-VDD): track 0.00 -> 3.17 mm
- net MISO_thermocouple: track 23.5 -> 26.4 mm
- net Net-(Q1-G): track 11.5 -> 9.54 mm

Commit message: limb circuit updates
Routing:
- net SDA_gyro: track 29.7 -> 29.0 mm
Other:
- board text added: "Gyroscope"
Changed lines of the file:
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@@
 		)
 		(property "Footprint" "21-0041B_8_MXM"
-			(at 0 0 360)
+			(at 0 0 0)
 			(layer "F.Fab")
 			(hide yes)
@@
 		)
 		(property "Datasheet" "MAX31855KASA+T"
-			(at 0 0 360)
+			(at 0 0 0)
 			(layer "F.Fab")
 			(hide yes)
@@
 		)
 		(property "Description" ""
-			(at 0 0 360)
+			(at 0 0 0)
 			(layer "F.Fab")
 			(hide yes)
@@
 		)
 		(fp_text user "*"
-			(at -2.97815 -3.5814 360)
+			(at -2.97815 -3.5814 0)
 			(layer "F.SilkS")
 			(effects
@@
 		)
 		(fp_text user "*"
-			(at -1.6129 -2.4257 360)
+			(at -1.6129 -2.4257 0)
 			(layer "F.Fab")
 			(effects
@@
 		(tags "LGA NoLead")
 		(property "Reference" "U2"
-			(at 0 -2.2 360)
+			(at 0 -2.2 0)
 			(layer "F.SilkS")
 			(effects
@@
 		)
 		(property "Value" "LSM6DSL"
-			(at 0 2.2 360)
+			(at 0 2.2 0)
 			(layer "F.Fab")
 			(effects
@@
 		)
 		(fp_text user "${REFERENCE}"
-			(at 0 0 360)
+			(at 0 0 0)
 			(layer "F.Fab")
 			(effects
@@
 		(layer "Edge.Cuts")
 	)
+	(gr_text "Gyroscope"
+		(at 119.5 138.5 0)
+		(layer "F.SilkS")
+		(effects
+			(font
+				(size 1 1)
+				(thickness 0.1)
+			)
+			(justify left bottom)
+		)
+	)
+	(gr_text_box "Exoskeleton Limb Circuit v0.1\n- Heating\n- Thermocouple\n- Gyroscope"
+		(start 152 136.5)
+		(end 172 147.5)
+		(layer "F.SilkS")
+		(effects
+			(font
+				(size 1 1)
+				(thickness 0.1)
+			)
+			(justify left top)
+		)
+		(border yes)
+		(stroke
+			(width 0.1)
+			(type solid)
+		)
+	)
 	(segment
 		(start 100.92 150.23)
@@
 	)
 	(segment
-		(start 128.1925 137.175)
-		(end 128.03 137.3375)
-		(width 0.2)
-		(layer "F.Cu")
-		(net 9)
-	)
-	(segment
 		(start 115.820635 135.635)
 		(end 113.620635 133.435)
@@
 	)
 	(segment
-		(start 128.6925 137.175)
-		(end 128.1925 137.175)
-		(width 0.2)
-		(layer "F.Cu")
-		(net 9)
-	)
-	(segment
 		(start 128.03 137.3375)
 		(end 126.3275 135.635)
@@
 		(min_thickness 0.25)
 		(filled_areas_thickness no)
-		(fill yes
+		(fill
 			(thermal_gap 0.5)
 			(thermal_bridge_width 0.5)

Commit message: Finished limb circuit board
Parts:
- removed R3: 10k, Resistor_SMD:R_0805_2012Metric
- removed the REF** at (170.0, 151.5)
- removed the REF** at (170.0, 109.5)
- removed the REF** at (93.5, 109.5)
- removed the REF** at (93.5, 151.5)
- added REF**: MountingHole_2.2mm_M2_DIN965_Pad, MountingHole:MountingHole_2.2mm_M2_DIN965_Pad, F.Cu at (115.5, 155.0)
- added REF**: MountingHole_2.2mm_M2_DIN965_Pad, MountingHole:MountingHole_2.2mm_M2_DIN965_Pad, F.Cu at (116.5, 107.0)
- moved A1 59.0 mm to (140.5, 152.5), turned to 180 degrees
- moved J3 49.2 mm to (106.7, 118.6), turned to 90 degrees
- moved J2 42.4 mm to (106.7, 153.1), turned to 90 degrees
- moved U1 36.1 mm to (115.5, 115.0), turned to 0 degrees
- moved C1 23.7 mm to (114.5, 130.0)
- moved C2 20.3 mm to (114.0, 134.5)
- moved J1 17.8 mm to (106.7, 135.8), turned to 90 degrees
- moved Q1 14.5 mm to (113.7, 141.1), turned to 0 degrees
- moved U2 10.8 mm to (120.0, 132.5)
- moved R1 8.50 mm to (116.9, 125.0), turned to 180 degrees
- moved R2 6.63 mm to (112.7, 125.0), turned to 0 degrees
Connections:
- U2 pad 1: SDA_gyro -> 3.3V_ard
- U2 pad 12: CS_gyro -> 3.3V_ard
Routing:
- net Net-(Q1-G): track 9.54 -> 71.9 mm
- net Net-(J3-Pin_2): track 44.8 -> 7.35 mm
- net Net-(J3-Pin_1): track 37.1 -> 7.35 mm
- net SDA_gyro: track 29.0 -> 8.80 mm
- net GND_16.4V: track 121.5 -> 104.2 mm
- net PWM_heater: track 38.2 -> 23.9 mm
- net SCL_gyro: track 23.5 -> 9.53 mm
- net Net-(U2-VDD): track 3.17 -> 8.72 mm
- net 3.3V_ard: track 43.2 -> 37.9 mm
- net GND_heater: track 18.1 -> 15.1 mm
- net CS_thermocouple: track 26.9 -> 23.9 mm
- net CLK: track 10.1 -> 7.05 mm
- net MISO_thermocouple: track 26.4 -> 23.3 mm
Other:
- board size 84.5 x 49.5 mm -> 56.5 x 56 mm
- board text added: "NANOTECH EXOSKELETON LIMB CIRCUIT V0.1"
- board text removed: "Gyroscope"
