File: Kicad Files/Limb Circuit/Limb_Circuit.kicad_sch (KiCad schematic)
At the start: 9 parts, among them J1 XT60_F_16.6V, J2 XT60_F_Heater, J3 XT60_F_Thermocouple, Q1 BUK9M52-40EX, U1 MAX31855KASA+T, U2 LSM6DSL

Commit message: Added gyroscope
Parts:
- added C1, C2: 0.1uF, Capacitor_SMD:C_0402_1005Metric, symbol Device:C_Small
- added R3: 10k, Resistor_SMD:R_0805_2012Metric, symbol Device:R_Small
Connections:
- net +3.3V: now also C1.1, R3.2; no longer U2.8 (VDD)
- net GND: now also U2.6 (GND), U2.7 (GND), C1.2, C2.2
- net SDA_gyro: now reaches A1.23 (A4)
- net SDA_gyro: now also U2.1 (SDO/SA0), U2.14 (SDA), R3.1
- net SCL_gyro: now reaches A1.24 (A5)
- net SCL_gyro: now also U2.13 (SCL)
- net CS_gyro: now reaches U2.12 (CS)
- new net: C2.1, U2.8 (VDD)
- no-connect marks 23 -> 25
Other:
- moved on the sheet: U2

Commit message: limb circuit updates
Parts:
- removed R3: 10k, Resistor_SMD:R_0805_2012Metric, symbol Device:R_Small
Connections:
- net +3.3V: now also U2.1 (SDO/SA0), U2.12 (CS)
- net CS_gyro: now also A1.7 (D4); no longer U2.12 (CS)
- net SDA_gyro: no longer U2.1 (SDO/SA0)
- no-connect marks 25 -> 24

Commit message: Finished limb circuit board
Connections:
- net CS_gyro: no longer names the net of A1.7 (D4)
- no-connect marks 24 -> 25
Changed lines of the file:
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@@
+	)
+	(no_connect
+		(at 86.36 110.49)
 	)
 	(no_connect
@@
 	(wire
 		(pts
-			(xy 80.01 110.49) (xy 86.36 110.49)
-		)
-		(stroke
-			(width 0)
-			(type default)
-		)
-	)
-	(wire
-		(pts
 			(xy 149.86 48.26) (xy 149.86 54.61)
 		)
@@
 				(hide yes)
 			)
-		)
-	)
-	(global_label "CS_gyro"
-		(shape input)
-		(at 80.01 110.49 180)
-		(fields_autoplaced yes)
-		(effects
-			(font
-				(size 1.27 1.27)
-			)
-			(justify right)
-		)
-		(property "Intersheetrefs" "${INTERSHEET_REFS}"
-			(at 69.5259 110.49 0)
-			(effects
-				(font
-					(size 1.27 1.27)
-				)
-				(justify right)
-				(hide yes)
-			)
